File: z9-console/sensor.kicad_sch (KiCad schematic)
At the start: 17 parts, among them U11 ST_SENSOR_2, U9 ISM330DHCX

Commit message: removed dil24
Parts:
- removed R24, R25, R26, R27: 10K, dnt:R_0402_1005Metric, symbol dnt_global:0402,10kΩ
- removed U11: ST_SENSOR_2, dnt:DIP-24_W15.24mm_Socket- nox, symbol dnt_global:ST_SENSOR_2
Connections:
- net +3.3V: no longer U9.11 (SDO_AUX), U9.2 (SDx), U9.3 (SCx)
- no-connect marks 3 -> 4
Other:
- moved on the sheet: C28
