File: z9-console/lcd.kicad_sch (KiCad schematic)
At the start: 15 parts, among them J2 LCD 3.2" 240x320 Conn_01x14_P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, J3 Conn_01x14_Pin, J4 Conn_01x04_Pin, J5 Conn_01x18_Pin, Q2 NPN, U2 TPS22919DCKR, U3 SN74LVC1G14DRLR, U4 XC6206PxxxMR

Commit message: Remove unused labels and wires from schematic SD Card junk
Connections:
- net SD_CS: no longer names the net of J4.1 (Pin_1)
- net SD_SCK: no longer names the net of J4.4 (Pin_4)
- net SD_SDI: no longer names the net of J4.3 (Pin_3)
- net SD_SDO: no longer names the net of J4.2 (Pin_2)
- no-connect marks 10 -> 14
Changed lines of the file:
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@@
+	)
+	(no_connect
+		(at 71.12 156.21)
+	)
+	(no_connect
+		(at 71.12 158.75)
+	)
+	(no_connect
+		(at 71.12 153.67)
+	)
+	(no_connect
+		(at 71.12 151.13)
 	)
 	(no_connect
@@
 	(wire
 		(pts
-			(xy 71.12 158.75) (xy 132.08 158.75)
-		)
-		(stroke
-			(width 0)
-			(type default)
-		)
-	)
-	(wire
-		(pts
 			(xy 71.12 63.5) (xy 76.2 63.5)
 		)
@@
 	(wire
 		(pts
-			(xy 71.12 156.21) (xy 132.08 156.21)
-		)
-		(stroke
-			(width 0)
-			(type default)
-		)
-	)
-	(wire
-		(pts
 			(xy 71.12 76.2) (xy 121.92 76.2)
 		)
@@
 	(wire
 		(pts
-			(xy 71.12 153.67) (xy 132.08 153.67)
-		)
-		(stroke
-			(width 0)
-			(type default)
-		)
-	)
-	(wire
-		(pts
 			(xy 71.12 73.66) (xy 132.08 73.66)
 		)
@@
 		(pts
 			(xy 104.14 22.86) (xy 97.79 22.86)
-		)
-		(stroke
-			(width 0)
-			(type default)
-		)
-	)
-	(wire
-		(pts
-			(xy 71.12 151.13) (xy 132.08 151.13)
 		)
 		(stroke
@@
 		)
 	)
-	(hierarchical_label "SD_SDI"
-		(shape input)
-		(at 132.08 156.21 0)
-		(effects
-			(font
-				(size 1.27 1.27)
-			)
-			(justify left)
-		)
-	)
 	(hierarchical_label "LCD_SCK"
 		(shape input)
@@
 		)
 	)
-	(hierarchical_label "SD_SDO"
-		(shape output)
-		(at 132.08 153.67 0)
-		(effects
-			(font
-				(size 1.27 1.27)
-			)
-			(justify left)
-		)
-	)
 	(hierarchical_label "LCD_RESET"
 		(shape input)
@@
 		(effects
 			(font
-				(size 1.27 1.27)
-			)
-			(justify left)
-		)
-	)
-	(hierarchical_label "SD_SCK"
-		(shape input)
-		(at 132.08 158.75 0)
-		(effects
-			(font
-				(size 1.27 1.27)
-			)
-			(justify left)
-		)
-	)
-	(hierarchical_label "SD_CS"
-		(shape input)
-		(at 132.08 151.13 0)
-		(effects
-			(font
