File: z9-shared/shared_isolated_can_ps.kicad_sch (KiCad schematic)
At the start: 3 parts, among them U976 B0505XT-1WR3

Commit message: Remove unused components and adjust annotation start number in project files
Parts:
- removed C976, C977: 10uF, dnt:C_0603_1608Metric, symbol dnt_global:0603,10uF,_25V
- removed U976: B0505XT-1WR3, dnt:B0505_Isolated_SMD, symbol dnt_global:B0505_Isolated_SMD
