File: z9-shared/shared_isolated_can.kicad_sch (KiCad schematic)
At the start: 9 parts, among them U951 ISO1042-Q1, U952 B0505XT-1WR3

Commit message: new fuse and ideal diode
Parts:
- C951, C953: symbol dnt_global:0603,100nF -> dnt_global:0603 100nF 50V X7R
Changed lines of the file:
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@@
 	)
 	(symbol
-		(lib_id "dnt_global:0603,100nF")
+		(lib_id "dnt_global:0603 100nF 50V X7R ")
 		(at 184.15 97.79 0)
 		(unit 1)
@@
 		(dnp no)
 		(property "Reference" "C953"
-			(at 185.42 97.79 90)
+			(at 186.182 96.122 0)
 			(effects
 				(font
@@
 		)
 		(property "Description" "50V 100nF X7R ±10% 0603 Multilayer Ceramic Capacitors MLCC - SMD/SMT ROHS"
-			(at 184.15 97.79 0)
+			(at 184.15 94.742 0)
 			(effects
 				(font
@@
 		)
 		(property "LCSC" "C14663"
-			(at 184.15 97.79 0)
+			(at 183.642 101.346 0)
 			(effects
 				(font
@@
 	)
 	(symbol
-		(lib_id "dnt_global:0603,100nF")
+		(lib_id "dnt_global:0603 100nF 50V X7R ")
 		(at 128.27 81.28 0)
 		(unit 1)
@@
 		(dnp no)
 		(property "Reference" "C951"
-			(at 129.54 80.01 90)
+			(at 130.302 79.612 0)
 			(effects
 				(font
@@
 		)
 		(property "Description" "50V 100nF X7R ±10% 0603 Multilayer Ceramic Capacitors MLCC - SMD/SMT ROHS"
-			(at 128.27 81.28 0)
+			(at 128.27 78.232 0)
 			(effects
 				(font
@@
 		)
 		(property "LCSC" "C14663"
-			(at 128.27 81.28 0)
-			(effects
-				(font
+			(at 127.762 84.836 0)
+			(effects
+				(font

Commit message: post 5v lay references lost
Connections:
- net +5V_ISO: no longer names the net of C952.1, C953.1, C955.1, U951.8 (VCC2), U952.5 (+VOUT)
Changed lines of the file:
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@@
-	)
-	(junction
-		(at 118.11 156.21)
-		(diameter 0)
-		(color 0 0 0 0)
 	)
 	(junction
@@
 	(wire
 		(pts
-			(xy 118.11 156.21) (xy 133.35 156.21)
-		)
-		(stroke
-			(width 0)
-			(type default)
-		)
-	)
-	(wire
-		(pts
 			(xy 114.3 166.37) (xy 118.11 166.37)
 		)
@@
 		)
 	)
-	(hierarchical_label "+5V_ISO"
-		(shape output)
-		(at 133.35 156.21 0)
-		(effects
-			(font
-				(size 1.27 1.27)
-				(thickness 0.1588)
-			)
-			(justify left)
-		)
-	)

Commit message: x
Parts:
- renumbered C954 to C56, C955 to C57, C951 to C58, C952 to C59, C953 to C60, JP951 to JP4, R951 to R76, U952 to U14, U951 to U15
Changed lines of the file:
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@@
 		(dnp no)
 		(fields_autoplaced yes)
-		(property "Reference" "#PWR0111"
+		(property "Reference" "#PWR0118"
 			(at 128.27 142.24 0)
 			(effects
@@
 		)
 		(property "Value" "GND"
-			(at 128.27 140.97 0)
-			(effects
-				(font
-					(size 1.27 1.27)
-				)
+			(at 130.81 137.1599 0)
+			(effects
+				(font
+					(size 1.27 1.27)
+				)
+				(justify left)
 			)
 		)
@@
 			(project "z9-pdm"
 				(path "/b643db5c-578e-4b48-aafc-cc4190db582a/2345b862-d871-4771-9bee-01079d71c128"
-					(reference "#PWR0111")
+					(reference "#PWR0118")
 					(unit 1)
 				)
@@
 		(on_board yes)
 		(dnp no)
-		(property "Reference" "C953"
+		(property "Reference" "C60"
 			(at 186.182 96.122 0)
 			(effects
@@
 			(project "z9-pdm"
 				(path "/b643db5c-578e-4b48-aafc-cc4190db582a/2345b862-d871-4771-9bee-01079d71c128"
-					(reference "C953")
+					(reference "C60")
 					(unit 1)
 				)
@@
 		(dnp no)
 		(fields_autoplaced yes)
-		(property "Reference" "#PWR0951"
+		(property "Reference" "#PWR0115"
 			(at 52.07 160.02 0)
 			(effects
@@
 		)
 		(property "Value" "+5V"
-			(at 52.07 151.13 0)
-			(effects
-				(font
-					(size 1.27 1.27)
-				)
+			(at 54.61 154.9399 0)
+			(effects
+				(font
+					(size 1.27 1.27)
+				)
+				(justify left)
 			)
 		)
@@
 			(project "z9-pdm"
 				(path "/b643db5c-578e-4b48-aafc-cc4190db582a/2345b862-d871-4771-9bee-01079d71c128"
-					(reference "#PWR0951")
+					(reference "#PWR0115")
 					(unit 1)
 				)
@@
 		(on_board yes)
 		(dnp no)
-		(property "Reference" "R951"
+		(property "Reference" "R76"
 			(at 190.5 73.66 90)
 			(effects
@@
 		(property "Description" "250mW Thick Film Resistors 200V ±100ppm/°C ±1% 120Ω 1206 Chip Resistor - Surface Mount ROHS"
 			(at 193.04 73.66 0)
-			(effects
-				(font
-					(size 1.27 1.27)
-				)
-				(hide yes)
-			)
-		)
-		(property "Order" ""
-			(at 193.04 73.66 90)
-			(effects
-				(font
-					(size 1.27 1.27)
-				)
-				(hide yes)
-			)
-		)
-		(property "PN" ""
-			(at 193.04 73.66 90)
-			(effects
-				(font
-					(size 1.27 1.27)
-				)
-				(hide yes)
-			)
-		)
-		(property "Part Number" ""
-			(at 193.04 73.66 90)
-			(effects
-				(font
-					(size 1.27 1.27)
-				)
-				(hide yes)
-			)
-		)
-		(property "Part#" ""
-			(at 193.04 73.66 90)
-			(effects
-				(font
-					(size 1.27 1.27)
-				)
-				(hide yes)
-			)
-		)
-		(property "Vendor" ""
-			(at 193.04 73.66 90)
-			(effects
-				(font
-					(size 1.27 1.27)
-				)
-				(hide yes)
-			)
-		)
-		(property "Voltage" ""
-			(at 193.04 73.66 90)
 			(effects
 				(font
@@
 			(project "z9-pdm"
 				(path "/b643db5c-578e-4b48-aafc-cc4190db582a/2345b862-d871-4771-9bee-01079d71c128"
-					(reference "R951")
+					(reference "R76")
 					(unit 1)
 				)
@@
 		(on_board yes)
 		(dnp no)
-		(property "Reference" "C951"
+		(property "Reference" "C58"
 			(at 130.302 79.612 0)
 			(effects
@@
 			(project "z9-pdm"
 				(path "/b643db5c-578e-4b48-aafc-cc4190db582a/2345b862-d871-4771-9bee-01079d71c128"
-					(reference "C951")
+					(reference "C58")
 					(unit 1)
 				)
@@
 		(on_board yes)
 		(dnp no)
-		(property "Reference" "C955"
+		(property "Reference" "C57"
 			(at 120.396 158.75 0)
 			(effects
@@
 		)
 		(property "Voltage Rated" "25V"
-			(at 120.904 162.052 0)
+			(at 120.142 162.0662 0)
 			(effects
 				(font
@@
 			(project "z9-pdm"
 				(path "/b643db5c-578e-4b48-aafc-cc4190db582a/2345b862-d871-4771-9bee-01079d71c128"
-					(reference "C955")
+					(reference "C57")
 					(unit 1)
 				)
@@
 		(on_board yes)
 		(dnp no)
-		(property "Reference" "C952"
+		(property "Reference" "C59"
 			(at 169.291 96.6216 0)
 			(effects
@@
 			(project "z9-pdm"
 				(path "/b643db5c-578e-4b48-aafc-cc4190db582a/2345b862-d871-4771-9bee-01079d71c128"
-					(reference "C952")
+					(reference "C59")
 					(unit 1)
 				)
@@
 		(dnp no)
 		(fields_autoplaced yes)
-		(property "Reference" "#PWR0110"
+		(property "Reference" "#PWR0117"
 			(at 78.74 77.47 0)
 			(effects
@@
 		)
 		(property "Value" "+3.3V"
-			(at 78.74 68.58 0)
-			(effects
-				(font
-					(size 1.27 1.27)
-				)
+			(at 81.28 72.3899 0)
+			(effects
+				(font
+					(size 1.27 1.27)
+				)
+				(justify left)
 			)
 		)
@@
 			(project "z9-pdm"
 				(path "/b643db5c-578e-4b48-aafc-cc4190db582a/2345b862-d871-4771-9bee-01079d71c128"
-					(reference "#PWR0110")
+					(reference "#PWR0117")
 					(unit 1)
 				)
@@
 		(on_board yes)
 		(dnp no)
-		(property "Reference" "C954"
+		(property "Reference" "C56"
 			(at 54.61 159.512 0)
 			(effects
@@
 		)
 		(property "Voltage Rated" "25V"
-			(at 55.626 162.814 0)
+			(at 54.102 162.0662 0)
 			(effects
 				(font
@@
 			(project "z9-pdm"
 				(path "/b643db5c-578e-4b48-aafc-cc4190db582a/2345b862-d871-4771-9bee-01079d71c128"
-					(reference "C954")
+					(reference "C56")
 					(unit 1)
 				)
@@
 		(dnp no)
 		(fields_autoplaced yes)
-		(property "Reference" "#PWR0952"
+		(property "Reference" "#PWR0116"
 			(at 52.07 184.15 0)
 			(effects
@@
 		)
 		(property "Value" "GND"
-			(at 52.07 182.88 0)
-			(effects
-				(font
-					(size 1.27 1.27)
-				)
+			(at 54.61 179.0699 0)
+			(effects
+				(font
+					(size 1.27 1.27)
+				)
+				(justify left)
 			)
 		)
@@
 			(project "z9-pdm"
 				(path "/b643db5c-578e-4b48-aafc-cc4190db582a/2345b862-d871-4771-9bee-01079d71c128"
-					(reference "#PWR0952")
+					(reference "#PWR0116")
 					(unit 1)
 				)
@@
 		(dnp no)
 		(fields_autoplaced yes)
-		(property "Reference" "U952"
+		(property "Reference" "U14"
 			(at 90.17 148.59 0)
 			(effects
@@
 			(project "z9-pdm"
 				(path "/b643db5c-578e-4b48-aafc-cc4190db582a/2345b862-d871-4771-9bee-01079d71c128"
-					(reference "U952")
+					(reference "U14")
 					(unit 1)
 				)
@@
 		(dnp yes)
 		(fields_autoplaced yes)
-		(property "Reference" "JP951"
+		(property "Reference" "JP4"
 			(at 195.58 64.7699 90)
 			(effects
@@
 		(property "Description" "Solder Jumper, 2-pole, closed/bridged"
 			(at 187.706 66.294 0)
-			(effects
-				(font
-					(size 1.27 1.27)
-				)
-				(hide yes)
-			)
-		)
-		(property "Order" ""
-			(at 193.04 66.04 90)
-			(effects
-				(font
-					(size 1.27 1.27)
-				)
-				(hide yes)
-			)
-		)
-		(property "PN" ""
-			(at 193.04 66.04 90)
-			(effects
-				(font
-					(size 1.27 1.27)
-				)
-				(hide yes)
-			)
-		)
-		(property "Part Number" ""
-			(at 193.04 66.04 90)
-			(effects
-				(font
-					(size 1.27 1.27)
-				)
-				(hide yes)
-			)
-		)
-		(property "Part#" ""
-			(at 193.04 66.04 90)
-			(effects
-				(font
-					(size 1.27 1.27)
-				)
-				(hide yes)
-			)
-		)
-		(property "Vendor" ""
-			(at 193.04 66.04 90)
-			(effects
-				(font
-					(size 1.27 1.27)
-				)
-				(hide yes)
-			)
-		)
-		(property "Voltage" ""
-			(at 193.04 66.04 90)
 			(effects
 				(font
@@
 			(project "z9-pdm"
 				(path "/b643db5c-578e-4b48-aafc-cc4190db582a/2345b862-d871-4771-9bee-01079d71c128"
-					(reference "JP951")
+					(reference "JP4")
 					(unit 1)
 				)
@@
 		(dnp no)
 		(fields_autoplaced yes)
-		(property "Reference" "U951"
+		(property "Reference" "U15"
 			(at 146.05 82.55 0)
 			(effects
@@
 			(project "z9-pdm"
 				(path "/b643db5c-578e-4b48-aafc-cc4190db582a/2345b862-d871-4771-9bee-01079d71c128"
-					(reference "U951")
-					(unit 1)
-				)
+					(reference "U15")
+					(unit 1)
+				)

Commit message: passes sch drc
Changed lines of the file:
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@@
 		)
 		(property "Value" "GND"
-			(at 130.81 137.1599 0)
-			(effects
-				(font
-					(size 1.27 1.27)
-				)
-				(justify left)
+			(at 128.27 140.97 0)
+			(effects
+				(font
+					(size 1.27 1.27)
+				)
 			)
 		)
@@
 		)
 		(property "Value" "+5V"
-			(at 54.61 154.9399 0)
-			(effects
-				(font
-					(size 1.27 1.27)
-				)
-				(justify left)
+			(at 52.07 151.13 0)
+			(effects
+				(font
+					(size 1.27 1.27)
+				)
 			)
 		)
@@
 		)
 		(property "Value" "+3.3V"
-			(at 81.28 72.3899 0)
-			(effects
-				(font
-					(size 1.27 1.27)
-				)
-				(justify left)
+			(at 78.74 68.58 0)
+			(effects
+				(font
+					(size 1.27 1.27)
+				)
 			)
 		)
@@
 		)
 		(property "Value" "GND"
-			(at 54.61 179.0699 0)
-			(effects
-				(font
-					(size 1.27 1.27)
-				)
-				(justify left)
-			)
-		)
+			(at 52.07 182.88 0)
+			(effects
+				(font
+					(size 1.27 1.27)
+				)
+			)
+		)

Commit message: core Refactor code structure for improved readability and maintainability
Parts:
- renumbered C58 to C951, C59 to C952, C60 to C953, C56 to C954, C57 to C955, JP4 to JP951, R76 to R951, U15 to U951, U14 to U952
Changed lines of the file:
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@@
 		(dnp no)
 		(fields_autoplaced yes)
-		(property "Reference" "#PWR0118"
+		(property "Reference" "#PWR0952"
 			(at 128.27 142.24 0)
 			(hide yes)
@@
 		(in_pos_files yes)
 		(dnp no)
-		(property "Reference" "C60"
+		(property "Reference" "C953"
 			(at 186.182 96.122 0)
 			(show_name no)
@@
 		(dnp no)
 		(fields_autoplaced yes)
-		(property "Reference" "#PWR0115"
+		(property "Reference" "#PWR0105"
 			(at 52.07 160.02 0)
 			(hide yes)
@@
 		(in_pos_files yes)
 		(dnp no)
-		(property "Reference" "R76"
+		(property "Reference" "R951"
 			(at 190.5 73.66 90)
 			(show_name no)
@@
 		(in_pos_files yes)
 		(dnp no)
-		(property "Reference" "C58"
+		(property "Reference" "C951"
 			(at 130.302 79.612 0)
 			(show_name no)
@@
 		(in_pos_files yes)
 		(dnp no)
-		(property "Reference" "C57"
+		(property "Reference" "C955"
 			(at 120.396 158.75 0)
 			(show_name no)
@@
 		(in_pos_files yes)
 		(dnp no)
-		(property "Reference" "C59"
+		(property "Reference" "C952"
 			(at 169.291 96.6216 0)
 			(show_name no)
@@
 		(dnp no)
 		(fields_autoplaced yes)
-		(property "Reference" "#PWR0117"
+		(property "Reference" "#PWR0951"
 			(at 78.74 77.47 0)
 			(hide yes)
@@
 		(in_pos_files yes)
 		(dnp no)
-		(property "Reference" "C56"
+		(property "Reference" "C954"
 			(at 54.61 159.512 0)
 			(show_name no)
@@
 		(dnp no)
 		(fields_autoplaced yes)
-		(property "Reference" "#PWR0116"
+		(property "Reference" "#PWR0106"
 			(at 52.07 184.15 0)
 			(hide yes)
@@
 		(dnp no)
 		(fields_autoplaced yes)
-		(property "Reference" "U14"
+		(property "Reference" "U952"
 			(at 90.17 148.59 0)
 			(show_name no)
@@
 		(dnp yes)
 		(fields_autoplaced yes)
-		(property "Reference" "JP4"
+		(property "Reference" "JP951"
 			(at 195.58 64.7699 90)
 			(show_name no)
@@
 		(dnp no)
 		(fields_autoplaced yes)
-		(property "Reference" "U15"
+		(property "Reference" "U951"
 			(at 146.05 82.55 0)
 			(show_name no)
