File: z9-shared/shared_ism330dhcx.kicad_sch (KiCad schematic)
At the start: 0 parts

Commit message: x
Parts:
- added C752: 100nF, PCM_JLCPCB:C_0402, symbol dnt_global:0402,100nF, 16V
- added C753: 10uF, dnt:C_0603_1608Metric, symbol dnt_global:0603,10uF,_25V
- added R754, R755, R756: 10K, dnt:R_0402_1005Metric, symbol dnt_global:0402,10kΩ
- added TP751: ISM_SDI, dnt:TestPoint_Pad_D1.0mm FP .6R, symbol Connector:TestPoint
- added TP752: ISM_INT1, dnt:TestPoint_Pad_D1.0mm FP .6R, symbol Connector:TestPoint
- added TP753: ISM_INT2, dnt:TestPoint_Pad_D1.0mm FP .6R, symbol Connector:TestPoint
- added TP754: ISM_SDO, dnt:TestPoint_Pad_D1.0mm FP .6R, symbol Connector:TestPoint
- added TP755: ISM3_SCK, dnt:TestPoint_Pad_D1.0mm FP .6R, symbol Connector:TestPoint
- added TP756: ISM_CS, dnt:TestPoint_Pad_D1.0mm FP .6R, symbol Connector:TestPoint
- added U751: ISM330DHCX, Package_LGA:LGA-14_3x2.5mm_P0.5mm_LayoutBorder3x4y, symbol dnt_global:ISM330DHCX
Connections:
- new net +3.3V: C752.1, C753.1, R754.2, U751.5 (VDDIO), U751.8 (VDD)
- new net GND: C752.2, C753.2, R755.1, R756.1, U751.6 (GND), U751.7 (GND)
- new net ISM_CS: R754.1, TP756.1, U751.12 (CS)
- new net ISM_INT1: R755.2, TP753.1, U751.4 (INT1)
- new net ISM_INT2: R756.2, TP752.1, U751.9 (INT2)
- new net ISM_SCK: TP755.1, U751.13 (SCL)
- new net ISM_SDI: TP751.1, U751.14 (SDA)
- new net ISM_SDO: TP754.1, U751.1 (SDO/SA0)
- no-connect marks 0 -> 4
Other:
- note added: "750 series"

Commit message: pre kicad update
Parts:
- renumbered C753 to C?, C752 to C?, R756 to R?, R755 to R?, R754 to R?, TP753 to TP?, TP756 to TP?, TP754 to TP?, TP755 to TP?, TP752 to TP?, TP751 to TP?, U751 to U?
Changed lines of the file:
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@@
 		(on_board yes)
 		(dnp no)
-		(property "Reference" "R756"
+		(property "Reference" "R?"
 			(at 144.272 115.57 90)
 			(effects
@@
 		(on_board yes)
 		(dnp no)
-		(property "Reference" "TP753"
+		(property "Reference" "TP?"
 			(at 100.965 110.49 90)
 			(effects
@@
 		(on_board yes)
 		(dnp no)
-		(property "Reference" "R755"
+		(property "Reference" "R?"
 			(at 139.192 115.57 90)
 			(effects
@@
 		(on_board yes)
 		(dnp no)
-		(property "Reference" "R754"
+		(property "Reference" "R?"
 			(at 123.19 43.688 0)
 			(effects
@@
 		(dnp no)
 		(fields_autoplaced yes)
-		(property "Reference" "#PWR0752"
+		(property "Reference" "#PWR?"
 			(at 95.25 26.67 0)
 			(effects
@@
 		(dnp no)
 		(fields_autoplaced yes)
-		(property "Reference" "U751"
+		(property "Reference" "U?"
 			(at 173.5933 85.09 0)
 			(effects
@@
 		(dnp no)
 		(fields_autoplaced yes)
-		(property "Reference" "#PWR0753"
+		(property "Reference" "#PWR?"
 			(at 205.74 151.13 0)
 			(effects
@@
 		(on_board yes)
 		(dnp no)
-		(property "Reference" "C753"
+		(property "Reference" "C?"
 			(at 208.661 38.2016 0)
 			(effects
@@
 		(on_board yes)
 		(dnp no)
-		(property "Reference" "TP756"
+		(property "Reference" "TP?"
 			(at 136.144 71.628 90)
 			(effects
@@
 		(on_board yes)
 		(dnp no)
-		(property "Reference" "TP754"
+		(property "Reference" "TP?"
 			(at 110.744 71.882 90)
 			(effects
@@
 		(on_board yes)
 		(dnp no)
-		(property "Reference" "C752"
+		(property "Reference" "C?"
 			(at 195.58 38.1 0)
 			(effects
@@
 		(on_board yes)
 		(dnp no)
-		(property "Reference" "TP755"
+		(property "Reference" "TP?"
 			(at 122.936 71.882 90)
 			(effects
@@
 		(on_board yes)
 		(dnp no)
-		(property "Reference" "TP752"
+		(property "Reference" "TP?"
 			(at 100.965 105.41 90)
 			(effects
@@
 		(on_board yes)
 		(dnp no)
-		(property "Reference" "TP751"
+		(property "Reference" "TP?"
 			(at 99.314 71.882 90)
 			(effects

Commit message: x
Parts:
- gave numbers to parts that had none: 12
Changed lines of the file:
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@@
 		(on_board yes)
 		(dnp no)
-		(property "Reference" "R?"
+		(property "Reference" "R756"
 			(at 144.272 115.57 90)
 			(effects
@@
 		(on_board yes)
 		(dnp no)
-		(property "Reference" "TP?"
+		(property "Reference" "TP753"
 			(at 100.965 110.49 90)
 			(effects
@@
 		(on_board yes)
 		(dnp no)
-		(property "Reference" "R?"
+		(property "Reference" "R755"
 			(at 139.192 115.57 90)
 			(effects
@@
 		(on_board yes)
 		(dnp no)
-		(property "Reference" "R?"
+		(property "Reference" "R754"
 			(at 123.19 43.688 0)
 			(effects
@@
 		(dnp no)
 		(fields_autoplaced yes)
-		(property "Reference" "#PWR?"
+		(property "Reference" "#PWR0752"
 			(at 95.25 26.67 0)
 			(effects
@@
 		(dnp no)
 		(fields_autoplaced yes)
-		(property "Reference" "U?"
+		(property "Reference" "U751"
 			(at 173.5933 85.09 0)
 			(effects
@@
 		(dnp no)
 		(fields_autoplaced yes)
-		(property "Reference" "#PWR?"
+		(property "Reference" "#PWR0753"
 			(at 205.74 151.13 0)
 			(effects
@@
 		(on_board yes)
 		(dnp no)
-		(property "Reference" "C?"
+		(property "Reference" "C753"
 			(at 208.661 38.2016 0)
 			(effects
@@
 		(on_board yes)
 		(dnp no)
-		(property "Reference" "TP?"
+		(property "Reference" "TP756"
 			(at 136.144 71.628 90)
 			(effects
@@
 		(on_board yes)
 		(dnp no)
-		(property "Reference" "TP?"
+		(property "Reference" "TP754"
 			(at 110.744 71.882 90)
 			(effects
@@
 		(on_board yes)
 		(dnp no)
-		(property "Reference" "C?"
+		(property "Reference" "C752"
 			(at 195.58 38.1 0)
 			(effects
@@
 		(on_board yes)
 		(dnp no)
-		(property "Reference" "TP?"
+		(property "Reference" "TP755"
 			(at 122.936 71.882 90)
 			(effects
@@
 		(on_board yes)
 		(dnp no)
-		(property "Reference" "TP?"
+		(property "Reference" "TP752"
 			(at 100.965 105.41 90)
 			(effects
@@
 		(on_board yes)
 		(dnp no)
-		(property "Reference" "TP?"
+		(property "Reference" "TP751"
 			(at 99.314 71.882 90)
 			(effects

Commit message: new fuse and ideal diode
Parts:
- C752: footprint PCM_JLCPCB:C_0402 -> dnt:C_0402_1005Metric
Changed lines of the file:
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@@
 		(dnp no)
 		(property "Reference" "C752"
-			(at 195.58 38.1 0)
+			(at 196.342 37.702 0)
 			(effects
 				(font
@@
 		)
 		(property "Value" "100nF"
-			(at 196.088 43.18 0)
+			(at 196.342 39.7482 0)
 			(effects
 				(font
-					(size 1.27 1.27)
+					(size 0.8 0.8)
 				)
 				(justify left)
 			)
 		)
-		(property "Footprint" "PCM_JLCPCB:C_0402"
+		(property "Footprint" "dnt:C_0402_1005Metric"
 			(at 192.532 39.37 90)
 			(effects
@@
 		)
 		(property "Voltage Rated" "16V"
-			(at 197.866 39.116 0)
+			(at 196.342 41.4162 0)
 			(effects
 				(font

Commit message: x
Parts:
- TP10: renamed from TP756; footprint dnt:TestPoint_Pad_D1.0mm FP .6R -> (none); Manufacturer DNP -> (none); Part # DNP -> (none); VEND DNP -> (none); VEND# DNP -> (none); now in the parts list
- TP5: renamed from TP751; footprint dnt:TestPoint_Pad_D1.0mm FP .6R -> (none); now in the parts list
- TP6: renamed from TP752; footprint dnt:TestPoint_Pad_D1.0mm FP .6R -> (none); now in the parts list
- TP7: renamed from TP753; footprint dnt:TestPoint_Pad_D1.0mm FP .6R -> (none); now in the parts list
- TP8: renamed from TP754; footprint dnt:TestPoint_Pad_D1.0mm FP .6R -> (none); Manufacturer DNP -> (none); Part # DNP -> (none); VEND DNP -> (none); VEND# DNP -> (none); now in the parts list
- TP9: renamed from TP755; footprint dnt:TestPoint_Pad_D1.0mm FP .6R -> (none); Manufacturer DNP -> (none); Part # DNP -> (none); VEND DNP -> (none); VEND# DNP -> (none); now in the parts list
- renumbered C752 to C53, C753 to C54, R754 to R68, R755 to R69, R756 to R70, U751 to U13

Commit message: passes sch drc
Parts:
- TP10, TP5, TP6, TP7, TP8, TP9: footprint (none) -> TestPoint:TestPoint_Pad_D1.0mm; symbol Connector:TestPoint -> dnt_global:TestPoint_Pad_D1.0mm
