File: z9-shared/shared_usbc.kicad_sch (KiCad schematic)
At the start: 10 parts, among them J18 USB_C_Receptacle_USB2.0_16P

Commit message: passes sch drc
Changed lines of the file:
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@@
 		)
 		(property "Value" "+5V"
-			(at 167.64 49.5299 0)
+			(at 165.1 45.72 0)
 			(effects
 				(font
 					(size 1.27 1.27)
 				)
-				(justify left)
 			)
 		)
