File: z9-shared/shared_buzzer.kicad_sch (KiCad schematic)
At the start: 9 parts, among them Q701 AO3400A

Commit message: pre kicad update
Parts:
- renumbered BZ701 to BZ?, C702 to C?, C703 to C?, C701 to C?, D701 to D?, FB701 to FB?, Q701 to Q?, R702 to R?, R701 to R?
Changed lines of the file:
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@@
 		(dnp no)
 		(fields_autoplaced yes)
-		(property "Reference" "FB701"
+		(property "Reference" "FB?"
 			(at 107.95 63.5507 0)
 			(effects
@@
 		(dnp no)
 		(fields_autoplaced yes)
-		(property "Reference" "Q701"
+		(property "Reference" "Q?"
 			(at 220.98 104.1399 0)
 			(effects
@@
 		(dnp no)
 		(fields_autoplaced yes)
-		(property "Reference" "D701"
+		(property "Reference" "D?"
 			(at 207.01 86.0424 0)
 			(effects
@@
 		(dnp no)
 		(fields_autoplaced yes)
-		(property "Reference" "#PWR0702"
+		(property "Reference" "#PWR0104"
 			(at 133.35 133.35 0)
 			(effects
@@
 		(dnp no)
 		(fields_autoplaced yes)
-		(property "Reference" "#PWR0704"
+		(property "Reference" "#PWR0102"
 			(at 194.31 133.35 0)
 			(effects
@@
 		(on_board yes)
 		(dnp no)
-		(property "Reference" "C702"
+		(property "Reference" "C?"
 			(at 147.32 87.63 90)
 			(effects
@@
 		(on_board yes)
 		(dnp no)
-		(property "Reference" "C703"
+		(property "Reference" "C?"
 			(at 196.85 83.82 90)
 			(effects
@@
 		(dnp no)
 		(fields_autoplaced yes)
-		(property "Reference" "BZ701"
+		(property "Reference" "BZ?"
 			(at 223.52 85.0899 0)
 			(effects
@@
 		(dnp no)
 		(fields_autoplaced yes)
-		(property "Reference" "#PWR0703"
+		(property "Reference" "#PWR0105"
 			(at 148.59 133.35 0)
 			(effects
@@
 		(dnp no)
 		(fields_autoplaced yes)
-		(property "Reference" "C701"
+		(property "Reference" "C?"
 			(at 135.89 83.8199 0)
 			(effects
@@
 		(on_board yes)
 		(dnp no)
-		(property "Reference" "R702"
+		(property "Reference" "R?"
 			(at 196.342 116.84 90)
 			(effects
@@
 		(dnp no)
 		(fields_autoplaced yes)
-		(property "Reference" "#PWR0701"
+		(property "Reference" "#PWR0103"
 			(at 104.14 52.07 0)
 			(effects
@@
 		(on_board yes)
 		(dnp no)
-		(property "Reference" "R701"
+		(property "Reference" "R?"
 			(at 189.23 107.95 90)
 			(effects
@@
 		(dnp no)
 		(fields_autoplaced yes)
-		(property "Reference" "#PWR0705"
+		(property "Reference" "#PWR0101"
 			(at 217.17 133.35 0)
 			(effects

Commit message: x
Parts:
- gave numbers to parts that had none: 9
Changed lines of the file:
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@@
 		(dnp no)
 		(fields_autoplaced yes)
-		(property "Reference" "FB?"
+		(property "Reference" "FB701"
 			(at 107.95 63.5507 0)
 			(effects
@@
 		(dnp no)
 		(fields_autoplaced yes)
-		(property "Reference" "Q?"
+		(property "Reference" "Q701"
 			(at 220.98 104.1399 0)
 			(effects
@@
 		(dnp no)
 		(fields_autoplaced yes)
-		(property "Reference" "D?"
+		(property "Reference" "D701"
 			(at 207.01 86.0424 0)
 			(effects
@@
 		(dnp no)
 		(fields_autoplaced yes)
-		(property "Reference" "#PWR0104"
+		(property "Reference" "#PWR0702"
 			(at 133.35 133.35 0)
 			(effects
@@
 		(dnp no)
 		(fields_autoplaced yes)
-		(property "Reference" "#PWR0102"
+		(property "Reference" "#PWR0704"
 			(at 194.31 133.35 0)
 			(effects
@@
 		(on_board yes)
 		(dnp no)
-		(property "Reference" "C?"
+		(property "Reference" "C702"
 			(at 147.32 87.63 90)
 			(effects
@@
 		(on_board yes)
 		(dnp no)
-		(property "Reference" "C?"
+		(property "Reference" "C703"
 			(at 196.85 83.82 90)
 			(effects
@@
 		(dnp no)
 		(fields_autoplaced yes)
-		(property "Reference" "BZ?"
+		(property "Reference" "BZ701"
 			(at 223.52 85.0899 0)
 			(effects
@@
 		(dnp no)
 		(fields_autoplaced yes)
-		(property "Reference" "#PWR0105"
+		(property "Reference" "#PWR0703"
 			(at 148.59 133.35 0)
 			(effects
@@
 		(dnp no)
 		(fields_autoplaced yes)
-		(property "Reference" "C?"
+		(property "Reference" "C701"
 			(at 135.89 83.8199 0)
 			(effects
@@
 		(on_board yes)
 		(dnp no)
-		(property "Reference" "R?"
+		(property "Reference" "R702"
 			(at 196.342 116.84 90)
 			(effects
@@
 		(dnp no)
 		(fields_autoplaced yes)
-		(property "Reference" "#PWR0103"
+		(property "Reference" "#PWR0701"
 			(at 104.14 52.07 0)
 			(effects
@@
 		(on_board yes)
 		(dnp no)
-		(property "Reference" "R?"
+		(property "Reference" "R701"
 			(at 189.23 107.95 90)
 			(effects
@@
 		(dnp no)
 		(fields_autoplaced yes)
-		(property "Reference" "#PWR0101"
+		(property "Reference" "#PWR0705"
 			(at 217.17 133.35 0)
 			(effects

Commit message: new fuse and ideal diode
Parts:
- C702, C703: symbol dnt_global:0603,100nF -> dnt_global:0603 100nF 50V X7R
Changed lines of the file:
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@@
 	)
 	(symbol
-		(lib_id "dnt_global:0603,100nF")
+		(lib_id "dnt_global:0603 100nF 50V X7R ")
 		(at 148.59 86.36 180)
 		(unit 1)
@@
 		(dnp no)
 		(property "Reference" "C702"
-			(at 147.32 87.63 90)
+			(at 146.558 88.028 0)
 			(effects
 				(font
@@
 		)
 		(property "Description" "50V 100nF X7R ±10% 0603 Multilayer Ceramic Capacitors MLCC - SMD/SMT ROHS"
-			(at 148.59 86.36 0)
+			(at 148.59 89.408 0)
 			(effects
 				(font
@@
 		)
 		(property "LCSC" "C14663"
-			(at 148.59 86.36 0)
+			(at 149.098 82.804 0)
 			(effects
 				(font
@@
 	)
 	(symbol
-		(lib_id "dnt_global:0603,100nF")
+		(lib_id "dnt_global:0603 100nF 50V X7R ")
 		(at 195.58 85.09 0)
 		(unit 1)
@@
 		(dnp no)
 		(property "Reference" "C703"
-			(at 196.85 83.82 90)
+			(at 197.612 83.422 0)
 			(effects
 				(font
@@
 		)
 		(property "Description" "50V 100nF X7R ±10% 0603 Multilayer Ceramic Capacitors MLCC - SMD/SMT ROHS"
-			(at 195.58 85.09 0)
+			(at 195.58 82.042 0)
 			(effects
 				(font
@@
 		)
 		(property "LCSC" "C14663"
-			(at 195.58 85.09 0)
-			(effects
-				(font
+			(at 195.072 88.646 0)
+			(effects
+				(font

Commit message: x
Parts:
- renumbered BZ701 to BZ2, C701 to C50, C702 to C51, C703 to C52, D701 to D32, FB701 to FB4, Q701 to Q3, R701 to R66, R702 to R67
Changed lines of the file:
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@@
 		(dnp no)
 		(fields_autoplaced yes)
-		(property "Reference" "FB701"
+		(property "Reference" "FB4"
 			(at 107.95 63.5507 0)
 			(effects
@@
 			(project "z9-pdm"
 				(path "/b643db5c-578e-4b48-aafc-cc4190db582a/c97401c5-7e03-4d93-a14f-f692468677b5"
-					(reference "FB701")
+					(reference "FB4")
 					(unit 1)
 				)
@@
 		(dnp no)
 		(fields_autoplaced yes)
-		(property "Reference" "Q701"
+		(property "Reference" "Q3"
 			(at 220.98 104.1399 0)
 			(effects
@@
 			(project "z9-pdm"
 				(path "/b643db5c-578e-4b48-aafc-cc4190db582a/c97401c5-7e03-4d93-a14f-f692468677b5"
-					(reference "Q701")
+					(reference "Q3")
 					(unit 1)
 				)
@@
 		(dnp no)
 		(fields_autoplaced yes)
-		(property "Reference" "D701"
+		(property "Reference" "D32"
 			(at 207.01 86.0424 0)
 			(effects
@@
 		)
 		(property "Reverse Leakage Current (Ir)" "500nA"
-			(at 204.47 87.63 0)
-			(effects
-				(font
-					(size 1.27 1.27)
-				)
-				(hide yes)
-			)
-		)
-		(property "Order" ""
-			(at 204.47 87.63 0)
-			(effects
-				(font
-					(size 1.27 1.27)
-				)
-				(hide yes)
-			)
-		)
-		(property "PN" ""
-			(at 204.47 87.63 0)
-			(effects
-				(font
-					(size 1.27 1.27)
-				)
-				(hide yes)
-			)
-		)
-		(property "Part Number" ""
-			(at 204.47 87.63 0)
-			(effects
-				(font
-					(size 1.27 1.27)
-				)
-				(hide yes)
-			)
-		)
-		(property "Part#" ""
-			(at 204.47 87.63 0)
-			(effects
-				(font
-					(size 1.27 1.27)
-				)
-				(hide yes)
-			)
-		)
-		(property "Vendor" ""
-			(at 204.47 87.63 0)
-			(effects
-				(font
-					(size 1.27 1.27)
-				)
-				(hide yes)
-			)
-		)
-		(property "Voltage" ""
 			(at 204.47 87.63 0)
 			(effects
@@
 			(project "z9-pdm"
 				(path "/b643db5c-578e-4b48-aafc-cc4190db582a/c97401c5-7e03-4d93-a14f-f692468677b5"
-					(reference "D701")
+					(reference "D32")
 					(unit 1)
 				)
@@
 		(dnp no)
 		(fields_autoplaced yes)
-		(property "Reference" "#PWR0702"
+		(property "Reference" "#PWR0101"
 			(at 133.35 133.35 0)
 			(effects
@@
 		)
 		(property "Value" "GND"
-			(at 133.35 132.08 0)
-			(effects
-				(font
-					(size 1.27 1.27)
-				)
+			(at 135.89 128.2699 0)
+			(effects
+				(font
+					(size 1.27 1.27)
+				)
+				(justify left)
 			)
 		)
@@
 			(project "z9-pdm"
 				(path "/b643db5c-578e-4b48-aafc-cc4190db582a/c97401c5-7e03-4d93-a14f-f692468677b5"
-					(reference "#PWR0702")
+					(reference "#PWR0101")
 					(unit 1)
 				)
@@
 		(dnp no)
 		(fields_autoplaced yes)
-		(property "Reference" "#PWR0704"
+		(property "Reference" "#PWR0103"
 			(at 194.31 133.35 0)
 			(effects
@@
 		)
 		(property "Value" "GND"
-			(at 194.31 132.08 0)
-			(effects
-				(font
-					(size 1.27 1.27)
-				)
+			(at 196.85 128.2699 0)
+			(effects
+				(font
+					(size 1.27 1.27)
+				)
+				(justify left)
 			)
 		)
@@
 			(project "z9-pdm"
 				(path "/b643db5c-578e-4b48-aafc-cc4190db582a/c97401c5-7e03-4d93-a14f-f692468677b5"
-					(reference "#PWR0704")
+					(reference "#PWR0103")
 					(unit 1)
 				)
@@
 		(on_board yes)
 		(dnp no)
-		(property "Reference" "C702"
+		(property "Reference" "C51"
 			(at 146.558 88.028 0)
 			(effects
@@
 			(project "z9-pdm"
 				(path "/b643db5c-578e-4b48-aafc-cc4190db582a/c97401c5-7e03-4d93-a14f-f692468677b5"
-					(reference "C702")
+					(reference "C51")
 					(unit 1)
 				)
@@
 		(on_board yes)
 		(dnp no)
-		(property "Reference" "C703"
+		(property "Reference" "C52"
 			(at 197.612 83.422 0)
 			(effects
@@
 			(project "z9-pdm"
 				(path "/b643db5c-578e-4b48-aafc-cc4190db582a/c97401c5-7e03-4d93-a14f-f692468677b5"
-					(reference "C703")
+					(reference "C52")
 					(unit 1)
 				)
@@
 		(dnp no)
 		(fields_autoplaced yes)
-		(property "Reference" "BZ701"
+		(property "Reference" "BZ2"
 			(at 223.52 85.0899 0)
 			(effects
@@
 			(project "z9-pdm"
 				(path "/b643db5c-578e-4b48-aafc-cc4190db582a/c97401c5-7e03-4d93-a14f-f692468677b5"
-					(reference "BZ701")
+					(reference "BZ2")
 					(unit 1)
 				)
@@
 		(dnp no)
 		(fields_autoplaced yes)
-		(property "Reference" "#PWR0703"
+		(property "Reference" "#PWR0102"
 			(at 148.59 133.35 0)
 			(effects
@@
 		)
 		(property "Value" "GND"
-			(at 148.59 132.08 0)
-			(effects
-				(font
-					(size 1.27 1.27)
-				)
+			(at 151.13 128.2699 0)
+			(effects
+				(font
+					(size 1.27 1.27)
+				)
+				(justify left)
 			)
 		)
@@
 			(project "z9-pdm"
 				(path "/b643db5c-578e-4b48-aafc-cc4190db582a/c97401c5-7e03-4d93-a14f-f692468677b5"
-					(reference "#PWR0703")
+					(reference "#PWR0102")
 					(unit 1)
 				)
@@
 		(dnp no)
 		(fields_autoplaced yes)
-		(property "Reference" "C701"
+		(property "Reference" "C50"
 			(at 135.89 83.8199 0)
 			(effects
@@
 			(project "z9-pdm"
 				(path "/b643db5c-578e-4b48-aafc-cc4190db582a/c97401c5-7e03-4d93-a14f-f692468677b5"
-					(reference "C701")
+					(reference "C50")
 					(unit 1)
 				)
@@
 		(on_board yes)
 		(dnp no)
-		(property "Reference" "R702"
+		(property "Reference" "R67"
 			(at 196.342 116.84 90)
 			(effects
@@
 			(project "z9-pdm"
 				(path "/b643db5c-578e-4b48-aafc-cc4190db582a/c97401c5-7e03-4d93-a14f-f692468677b5"
-					(reference "R702")
+					(reference "R67")
 					(unit 1)
 				)
@@
 		(dnp no)
 		(fields_autoplaced yes)
-		(property "Reference" "#PWR0701"
+		(property "Reference" "#PWR0100"
 			(at 104.14 52.07 0)
 			(effects
@@
 		)
 		(property "Value" "+3.3V"
-			(at 104.14 43.18 0)
-			(effects
-				(font
-					(size 1.27 1.27)
-				)
+			(at 106.68 46.9899 0)
+			(effects
+				(font
+					(size 1.27 1.27)
+				)
+				(justify left)
 			)
 		)
@@
 			(project "z9-pdm"
 				(path "/b643db5c-578e-4b48-aafc-cc4190db582a/c97401c5-7e03-4d93-a14f-f692468677b5"
-					(reference "#PWR0701")
+					(reference "#PWR0100")
 					(unit 1)
 				)
@@
 		(on_board yes)
 		(dnp no)
-		(property "Reference" "R701"
+		(property "Reference" "R66"
 			(at 189.23 107.95 90)
 			(effects
@@
 			(project "z9-pdm"
 				(path "/b643db5c-578e-4b48-aafc-cc4190db582a/c97401c5-7e03-4d93-a14f-f692468677b5"
-					(reference "R701")
+					(reference "R66")
 					(unit 1)
 				)
@@
 		(dnp no)
 		(fields_autoplaced yes)
-		(property "Reference" "#PWR0705"
+		(property "Reference" "#PWR0104"
 			(at 217.17 133.35 0)
 			(effects
@@
 		)
 		(property "Value" "GND"
-			(at 217.17 132.08 0)
-			(effects
-				(font
-					(size 1.27 1.27)
-				)
+			(at 219.71 128.2699 0)
+			(effects
+				(font
+					(size 1.27 1.27)
+				)
+				(justify left)
 			)
 		)
@@
 			(project "z9-pdm"
 				(path "/b643db5c-578e-4b48-aafc-cc4190db582a/c97401c5-7e03-4d93-a14f-f692468677b5"
-					(reference "#PWR0705")
-					(unit 1)
-				)
+					(reference "#PWR0104")
+					(unit 1)
+				)

Commit message: passes sch drc
Changed lines of the file:
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@@
 		)
 		(property "Value" "GND"
-			(at 135.89 128.2699 0)
-			(effects
-				(font
-					(size 1.27 1.27)
-				)
-				(justify left)
+			(at 133.35 132.08 0)
+			(effects
+				(font
+					(size 1.27 1.27)
+				)
 			)
 		)
@@
 		)
 		(property "Value" "GND"
-			(at 196.85 128.2699 0)
-			(effects
-				(font
-					(size 1.27 1.27)
-				)
-				(justify left)
+			(at 194.31 132.08 0)
+			(effects
+				(font
+					(size 1.27 1.27)
+				)
 			)
 		)
@@
 		)
 		(property "Value" "GND"
-			(at 151.13 128.2699 0)
-			(effects
-				(font
-					(size 1.27 1.27)
-				)
-				(justify left)
+			(at 148.59 132.08 0)
+			(effects
+				(font
+					(size 1.27 1.27)
+				)
 			)
 		)
@@
 		)
 		(property "Value" "+3.3V"
-			(at 106.68 46.9899 0)
-			(effects
-				(font
-					(size 1.27 1.27)
-				)
-				(justify left)
+			(at 104.14 43.18 0)
+			(effects
+				(font
+					(size 1.27 1.27)
+				)
 			)
 		)
@@
 		)
 		(property "Value" "GND"
-			(at 219.71 128.2699 0)
-			(effects
-				(font
-					(size 1.27 1.27)
-				)
-				(justify left)
-			)
-		)
+			(at 217.17 132.08 0)
+			(effects
+				(font
+					(size 1.27 1.27)
+				)
+			)
+		)

Commit message: kicad: migrate z9-pdm, z9-console and z9-shared projects to KiCad 10
Parts:
- FB4: value ~ -> (none)

Commit message: core Refactor code structure for improved readability and maintainability
Parts:
- renumbered BZ2 to BZ701, C50 to C701, C51 to C702, C52 to C703, D32 to D701, FB4 to FB701, Q3 to Q701, R66 to R701, R67 to R702
Changed lines of the file:
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@@
 		(dnp no)
 		(fields_autoplaced yes)
-		(property "Reference" "FB4"
+		(property "Reference" "FB701"
 			(at 107.95 63.5507 0)
 			(show_name no)
@@
 				)
 			)
-			(project ""
+			(project "z9-console"
 				(path "/8d063f79-9282-4820-bcf4-1ff3c006cf08/f06e6e31-c68d-491a-ad1f-dc0bf57e1d1a"
 					(reference "FB701")
@@
 		(dnp no)
 		(fields_autoplaced yes)
-		(property "Reference" "Q3"
+		(property "Reference" "Q701"
 			(at 220.98 104.1399 0)
 			(show_name no)
@@
 		(dnp no)
 		(fields_autoplaced yes)
-		(property "Reference" "D32"
+		(property "Reference" "D701"
 			(at 207.01 86.0424 0)
 			(show_name no)
@@
 		(dnp no)
 		(fields_autoplaced yes)
-		(property "Reference" "#PWR0101"
+		(property "Reference" "#PWR0702"
 			(at 133.35 133.35 0)
 			(hide yes)
@@
 		(dnp no)
 		(fields_autoplaced yes)
-		(property "Reference" "#PWR0103"
+		(property "Reference" "#PWR0704"
 			(at 194.31 133.35 0)
 			(hide yes)
@@
 		(in_pos_files yes)
 		(dnp no)
-		(property "Reference" "C51"
+		(property "Reference" "C702"
 			(at 146.558 88.028 0)
 			(show_name no)
@@
 		(in_pos_files yes)
 		(dnp no)
-		(property "Reference" "C52"
+		(property "Reference" "C703"
 			(at 197.612 83.422 0)
 			(show_name no)
@@
 		(dnp no)
 		(fields_autoplaced yes)
-		(property "Reference" "BZ2"
+		(property "Reference" "BZ701"
 			(at 223.52 85.0899 0)
 			(show_name no)
@@
 		(dnp no)
 		(fields_autoplaced yes)
-		(property "Reference" "#PWR0102"
+		(property "Reference" "#PWR0703"
 			(at 148.59 133.35 0)
 			(hide yes)
@@
 		(dnp no)
 		(fields_autoplaced yes)
-		(property "Reference" "C50"
+		(property "Reference" "C701"
 			(at 135.89 83.8199 0)
 			(show_name no)
@@
 				)
 			)
-			(project ""
+			(project "z9-console"
 				(path "/8d063f79-9282-4820-bcf4-1ff3c006cf08/f06e6e31-c68d-491a-ad1f-dc0bf57e1d1a"
 					(reference "C701")
@@
 		(in_pos_files yes)
 		(dnp no)
-		(property "Reference" "R67"
+		(property "Reference" "R702"
 			(at 196.342 116.84 90)
 			(show_name no)
@@
 		(dnp no)
 		(fields_autoplaced yes)
-		(property "Reference" "#PWR0100"
+		(property "Reference" "#PWR0701"
 			(at 104.14 52.07 0)
 			(hide yes)
@@
 				)
 			)
-			(project ""
+			(project "z9-console"
 				(path "/8d063f79-9282-4820-bcf4-1ff3c006cf08/f06e6e31-c68d-491a-ad1f-dc0bf57e1d1a"
 					(reference "#PWR0701")
@@
 		(in_pos_files yes)
 		(dnp no)
-		(property "Reference" "R66"
+		(property "Reference" "R701"
 			(at 189.23 107.95 90)
 			(show_name no)
@@
 		(dnp no)
 		(fields_autoplaced yes)
-		(property "Reference" "#PWR0104"
+		(property "Reference" "#PWR0705"
 			(at 217.17 133.35 0)
 			(hide yes)
