File: z9-pdm/vn9e30.kicad_sch (KiCad schematic)
At the start: 3 parts, among them U5 VN9E30F

Commit message: vipower fixes etc
Parts:
- added C704: 100nF, dnt:C_0603_1608Metric, symbol dnt_global:0603,100nF
- added R703: 150Ω, dnt:R_0603_1608Metric, symbol dnt_global:0603,150Ω
Connections:
- net +3.3V: now also R703.1; no longer U5.16 (VDD)
- net GND: now also C704.2
- net +12V renamed +12V_VIPOWER
- net +12V_VIPOWER: now also C704.1
- new net: R703.2, U5.16 (VDD)
