File: z9-pdm/vn9e30.kicad_sch (KiCad schematic)
At the start: 5 parts, among them U5 VN9E30F

Commit message: routing
Parts:
- removed R23: 2.7kΩ, PCM_JLCPCB:R_0603, symbol PCM_JLCPCB-Resistors:0603,2.7kΩ
Connections:
- net CS: now also U5.12 (CSN)

Commit message: new fuse and ideal diode
Parts:
- C704: symbol dnt_global:0603,100nF -> dnt_global:0603 100nF 50V X7R
Changed lines of the file:
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@@
 	)
 	(symbol
-		(lib_id "dnt_global:0603,100nF")
+		(lib_id "dnt_global:0603 100nF 50V X7R ")
 		(at 170.18 46.99 0)
 		(unit 1)
@@
 		)
 		(property "Description" "50V 100nF X7R ±10% 0603 Multilayer Ceramic Capacitors MLCC - SMD/SMT ROHS"
-			(at 170.18 46.99 0)
+			(at 170.18 43.942 0)
 			(effects
 				(font
@@
 		)
 		(property "LCSC" "C14663"
-			(at 170.18 46.99 0)
+			(at 169.672 50.546 0)
 			(effects
 				(font

Commit message: x
Parts:
- U2: renamed from U5; value VN9E30F -> VN9E30FTR; LCSC (none) -> C3225491
- renumbered C704 to C2, R703 to R2, R24 to R3
Changed lines of the file:
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@@
 	)
 	(junction
-		(at 101.6 71.12)
+		(at 101.6 78.74)
 		(diameter 0)
 		(color 0 0 0 0)
@@
 	(wire
 		(pts
-			(xy 83.82 71.12) (xy 101.6 71.12)
+			(xy 95.25 78.74) (xy 101.6 78.74)
 		)
 		(stroke
@@
 	(wire
 		(pts
-			(xy 83.82 67.31) (xy 83.82 71.12)
+			(xy 95.25 74.93) (xy 95.25 78.74)
 		)
 		(stroke
@@
 	(wire
 		(pts
-			(xy 101.6 71.12) (xy 101.6 111.76)
+			(xy 101.6 78.74) (xy 101.6 111.76)
 		)
 		(stroke
@@
 	(wire
 		(pts
-			(xy 157.48 39.37) (xy 170.18 39.37)
+			(xy 101.6 39.37) (xy 170.18 39.37)
 		)
 		(stroke
@@
 	(wire
 		(pts
-			(xy 101.6 64.77) (xy 101.6 71.12)
+			(xy 101.6 64.77) (xy 101.6 78.74)
 		)
 		(stroke
@@
 	(wire
 		(pts
-			(xy 157.48 36.83) (xy 157.48 39.37)
+			(xy 101.6 36.83) (xy 101.6 39.37)
 		)
 		(stroke
@@
 		(dnp no)
 		(fields_autoplaced yes)
-		(property "Reference" "#PWR038"
+		(property "Reference" "#PWR05"
 			(at 101.6 130.81 0)
 			(effects
@@
 		)
 		(property "Value" "GND"
-			(at 101.6 129.54 0)
-			(effects
-				(font
-					(size 1.27 1.27)
-				)
+			(at 104.14 125.7299 0)
+			(effects
+				(font
+					(size 1.27 1.27)
+				)
+				(justify left)
+				(hide yes)
 			)
 		)
@@
 			(project "z9-pdm-pcb"
 				(path "/b643db5c-578e-4b48-aafc-cc4190db582a/cd2147da-2530-4471-81dd-8f7a12e86f84/2bb75966-61f7-4749-a1a9-a4113474d2c6"
-					(reference "#PWR038")
+					(reference "#PWR05")
 					(unit 1)
 				)
 				(path "/b643db5c-578e-4b48-aafc-cc4190db582a/cd2147da-2530-4471-81dd-8f7a12e86f84/87b05001-00dc-4343-8786-c48b8f2631a1"
-					(reference "#PWR040")
+					(reference "#PWR021")
 					(unit 1)
 				)
@@
 		(dnp no)
 		(fields_autoplaced yes)
-		(property "Reference" "C704"
+		(property "Reference" "C2"
 			(at 172.72 44.4499 0)
 			(effects
@@
 			(project ""
 				(path "/b643db5c-578e-4b48-aafc-cc4190db582a/cd2147da-2530-4471-81dd-8f7a12e86f84/2bb75966-61f7-4749-a1a9-a4113474d2c6"
-					(reference "C704")
+					(reference "C2")
 					(unit 1)
 				)
 				(path "/b643db5c-578e-4b48-aafc-cc4190db582a/cd2147da-2530-4471-81dd-8f7a12e86f84/87b05001-00dc-4343-8786-c48b8f2631a1"
-					(reference "C705")
+					(reference "C10")
 					(unit 1)
 				)
@@
 		(on_board yes)
 		(dnp no)
-		(property "Reference" "R24"
+		(property "Reference" "R3"
 			(at 118.11 109.22 90)
 			(effects
@@
 			)
 		)
-		(property "Order" ""
-			(at 123.19 109.22 90)
-			(effects
-				(font
-					(size 1.27 1.27)
-				)
-				(hide yes)
-			)
-		)
-		(property "PN" ""
-			(at 123.19 109.22 90)
-			(effects
-				(font
-					(size 1.27 1.27)
-				)
-				(hide yes)
-			)
-		)
-		(property "Part Number" ""
-			(at 123.19 109.22 90)
-			(effects
-				(font
-					(size 1.27 1.27)
-				)
-				(hide yes)
-			)
-		)
-		(property "Part#" ""
-			(at 123.19 109.22 90)
-			(effects
-				(font
-					(size 1.27 1.27)
-				)
-				(hide yes)
-			)
-		)
-		(property "Vendor" ""
-			(at 123.19 109.22 90)
-			(effects
-				(font
-					(size 1.27 1.27)
-				)
-				(hide yes)
-			)
-		)
-		(property "Voltage" ""
-			(at 123.19 109.22 90)
-			(effects
-				(font
-					(size 1.27 1.27)
-				)
-				(hide yes)
-			)
-		)
 		(pin "1"
 		)
@@
 			(project "z9-pdm-pcb"
 				(path "/b643db5c-578e-4b48-aafc-cc4190db582a/cd2147da-2530-4471-81dd-8f7a12e86f84/2bb75966-61f7-4749-a1a9-a4113474d2c6"
-					(reference "R24")
+					(reference "R3")
 					(unit 1)
 				)
 				(path "/b643db5c-578e-4b48-aafc-cc4190db582a/cd2147da-2530-4471-81dd-8f7a12e86f84/87b05001-00dc-4343-8786-c48b8f2631a1"
-					(reference "R13")
+					(reference "R11")
 					(unit 1)
 				)
@@
 	(symbol
 		(lib_id "power:PWR_FLAG")
-		(at 83.82 67.31 0)
+		(at 95.25 74.93 0)
 		(unit 1)
 		(exclude_from_sim no)
@@
 		(dnp no)
 		(fields_autoplaced yes)
-		(property "Reference" "#FLG0702"
-			(at 83.82 65.405 0)
+		(property "Reference" "#FLG02"
+			(at 95.25 73.025 0)
 			(effects
 				(font
@@
 		)
 		(property "Value" "PWR_FLAG"
-			(at 83.82 62.23 0)
-			(effects
-				(font
-					(size 1.27 1.27)
-				)
+			(at 97.79 73.6599 0)
+			(effects
+				(font
+					(size 1.27 1.27)
+				)
+				(justify left)
+				(hide yes)
 			)
 		)
 		(property "Footprint" ""
-			(at 83.82 67.31 0)
+			(at 95.25 74.93 0)
 			(effects
 				(font
@@
 		)
 		(property "Datasheet" "~"
-			(at 83.82 67.31 0)
+			(at 95.25 74.93 0)
 			(effects
 				(font
@@
 		)
 		(property "Description" "Special symbol for telling ERC where power comes from"
-			(at 83.82 67.31 0)
+			(at 95.25 74.93 0)
 			(effects
 				(font
@@
 			(project ""
 				(path "/b643db5c-578e-4b48-aafc-cc4190db582a/cd2147da-2530-4471-81dd-8f7a12e86f84/2bb75966-61f7-4749-a1a9-a4113474d2c6"
-					(reference "#FLG0702")
+					(reference "#FLG02")
 					(unit 1)
 				)
 				(path "/b643db5c-578e-4b48-aafc-cc4190db582a/cd2147da-2530-4471-81dd-8f7a12e86f84/87b05001-00dc-4343-8786-c48b8f2631a1"
-					(reference "#FLG0703")
+					(reference "#FLG06")
 					(unit 1)
 				)
@@
 		(on_board yes)
 		(dnp no)
-		(property "Reference" "#PWR14"
+		(property "Reference" "#PWR04"
 			(at 101.6 55.88 0)
 			(effects
@@
 			(project "z9-pdm-pcb"
 				(path "/b643db5c-578e-4b48-aafc-cc4190db582a/cd2147da-2530-4471-81dd-8f7a12e86f84/2bb75966-61f7-4749-a1a9-a4113474d2c6"
-					(reference "#PWR14")
+					(reference "#PWR04")
 					(unit 1)
 				)
 				(path "/b643db5c-578e-4b48-aafc-cc4190db582a/cd2147da-2530-4471-81dd-8f7a12e86f84/87b05001-00dc-4343-8786-c48b8f2631a1"
-					(reference "#PWR36")
+					(reference "#PWR020")
 					(unit 1)
 				)
@@
 		(on_board yes)
 		(dnp no)
-		(property "Reference" "R703"
-			(at 104.14 60.9599 0)
+		(property "Reference" "R2"
+			(at 102.87 60.706 0)
 			(effects
 				(font
@@
 		)
 		(property "Value" "150Ω"
-			(at 97.028 59.436 90)
+			(at 98.552 60.452 0)
 			(do_not_autoplace yes)
 			(effects
@@
 			(project ""
 				(path "/b643db5c-578e-4b48-aafc-cc4190db582a/cd2147da-2530-4471-81dd-8f7a12e86f84/2bb75966-61f7-4749-a1a9-a4113474d2c6"
-					(reference "R703")
+					(reference "R2")
 					(unit 1)
 				)
 				(path "/b643db5c-578e-4b48-aafc-cc4190db582a/cd2147da-2530-4471-81dd-8f7a12e86f84/87b05001-00dc-4343-8786-c48b8f2631a1"
-					(reference "R704")
+					(reference "R10")
 					(unit 1)
 				)
@@
 		(dnp no)
 		(fields_autoplaced yes)
-		(property "Reference" "U5"
+		(property "Reference" "U2"
 			(at 157.48 63.5 0)
 			(effects
@@
 			)
 		)
-		(property "Value" "VN9E30F"
+		(property "Value" "VN9E30FTR"
 			(at 157.48 66.04 0)
 			(effects
@@
 			)
 		)
-		(property "Order" ""
+		(property "LCSC" "C3225491"
 			(at 132.08 73.66 0)
 			(effects
@@
 			)
 		)
-		(property "PN" ""
-			(at 132.08 73.66 0)
-			(effects
-				(font
-					(size 1.27 1.27)
-				)
-				(hide yes)
-			)
-		)
-		(property "Part Number" ""
-			(at 132.08 73.66 0)
-			(effects
-				(font
-					(size 1.27 1.27)
-				)
-				(hide yes)
-			)
-		)
-		(property "Part#" ""
-			(at 132.08 73.66 0)
-			(effects
-				(font
-					(size 1.27 1.27)
-				)
-				(hide yes)
-			)
-		)
-		(property "Vendor" ""
-			(at 132.08 73.66 0)
-			(effects
-				(font
-					(size 1.27 1.27)
-				)
-				(hide yes)
-			)
-		)
-		(property "Voltage" ""
-			(at 132.08 73.66 0)
-			(effects
-				(font
-					(size 1.27 1.27)
-				)
-				(hide yes)
-			)
-		)
 		(pin "16"
 		)
@@
 		)
 		(instances
-			(project "z9-pdm-pcb"
+			(project ""
+				(path "/b643db5c-578e-4b48-aafc-cc4190db582a/651fe70f-48a4-454d-84e2-56b28624b7c9"
+					(reference "U2")
+					(unit 1)
+				)
 				(path "/b643db5c-578e-4b48-aafc-cc4190db582a/cd2147da-2530-4471-81dd-8f7a12e86f84/2bb75966-61f7-4749-a1a9-a4113474d2c6"
+					(reference "U2")
+					(unit 1)
+				)
+				(path "/b643db5c-578e-4b48-aafc-cc4190db582a/cd2147da-2530-4471-81dd-8f7a12e86f84/87b05001-00dc-4343-8786-c48b8f2631a1"
 					(reference "U5")
-					(unit 1)
-				)
-				(path "/b643db5c-578e-4b48-aafc-cc4190db582a/cd2147da-2530-4471-81dd-8f7a12e86f84/87b05001-00dc-4343-8786-c48b8f2631a1"
-					(reference "U4")
 					(unit 1)
 				)
@@
 	(symbol
 		(lib_id "power:+12V")
-		(at 157.48 36.83 0)
+		(at 101.6 36.83 0)
 		(unit 1)
 		(exclude_from_sim no)
@@
 		(on_board yes)
 		(dnp no)
-		(property "Reference" "#PWR041"
-			(at 157.48 40.64 0)
+		(property "Reference" "#PWR06"
+			(at 101.6 40.64 0)
 			(effects
 				(font
@@
 		)
 		(property "Value" "+12V_VIPOWER"
-			(at 157.48 33.274 0)
+			(at 101.6 33.274 0)
 			(effects
 				(font
@@
 		)
 		(property "Footprint" ""
-			(at 157.48 36.83 0)
+			(at 101.6 36.83 0)
 			(effects
 				(font
@@
 		)
 		(property "Datasheet" ""
-			(at 157.48 36.83 0)
+			(at 101.6 36.83 0)
 			(effects
 				(font
@@
 		)
 		(property "Description" "Power symbol creates a global label with name \"+12V\""
-			(at 157.48 36.83 0)
+			(at 101.6 36.83 0)
 			(effects
 				(font
@@
 			(project "z9-pdm-pcb"
 				(path "/b643db5c-578e-4b48-aafc-cc4190db582a/cd2147da-2530-4471-81dd-8f7a12e86f84/2bb75966-61f7-4749-a1a9-a4113474d2c6"
-					(reference "#PWR041")
+					(reference "#PWR06")
 					(unit 1)
 				)
 				(path "/b643db5c-578e-4b48-aafc-cc4190db582a/cd2147da-2530-4471-81dd-8f7a12e86f84/87b05001-00dc-4343-8786-c48b8f2631a1"
-					(reference "#PWR045")
+					(reference "#PWR022")
 					(unit 1)
 				)
@@
 		(dnp no)
 		(fields_autoplaced yes)
-		(property "Reference" "#PWR0711"
+		(property "Reference" "#PWR07"
 			(at 170.18 57.15 0)
 			(effects
@@
 		)
 		(property "Value" "GND"
-			(at 170.18 55.88 0)
-			(effects
-				(font
-					(size 1.27 1.27)
-				)
+			(at 172.72 52.0699 0)
+			(effects
+				(font
+					(size 1.27 1.27)
+				)
+				(justify left)
+				(hide yes)
 			)
 		)
@@
 			(project "z9-pdm"
 				(path "/b643db5c-578e-4b48-aafc-cc4190db582a/cd2147da-2530-4471-81dd-8f7a12e86f84/2bb75966-61f7-4749-a1a9-a4113474d2c6"
-					(reference "#PWR0711")
+					(reference "#PWR07")
 					(unit 1)
 				)
 				(path "/b643db5c-578e-4b48-aafc-cc4190db582a/cd2147da-2530-4471-81dd-8f7a12e86f84/87b05001-00dc-4343-8786-c48b8f2631a1"
-					(reference "#PWR0712")
-					(unit 1)
-				)
+					(reference "#PWR023")
+					(unit 1)
+				)
