File: z9-pdm/stm32.kicad_sch (KiCad schematic)
At the start: 56 parts, among them J4 Conn_ST_STDC14, J5 DF40HC3.0-100DS-0.4V51, J7 Conn_TagConnect_2070, SW1 Tactile Button, 160gf, SW2 Tactile Button, 160gf, U3 STM32F427V_G-I_Tx, X1 8MHz 20pF

Commit message: Update DNP property for J4 connector and correct footprint reference in STM32 schematic
Parts:
- J4: footprint dnt:SAMTEC_FTSH-107-01-F-DV-K-Fix -> dnt:Conn_SAMTEC_FTSH-107-01-F-DV-K-Fix; now fitted

Commit message: x
Parts:
- D14, D5: LCSC (none) -> C2290
