File: z9-pdm/stm32.kicad_sch (KiCad schematic)
At the start: 33 parts, among them J2 Conn_ST_STDC14, J3 Conn_TagConnect_2070, J4 DF40HC(3.0)-100DS-0.4V(51), SW2 Tactile Button, 160gf, SW3 Tactile Button, 160gf, U6 STM32F427V_G-I_Tx, X2 8MHz 20pF

Commit message: z9-pdm: rename 12V net label and add wire connections
Connections:
- net SPI1_CS is gone; now on net SPI3_CS: U6.33 (PC4)
Changed lines of the file:
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@@
 (kicad_sch
-	(version 20250114)
+	(version 20260306)
 	(generator "eeschema")
-	(generator_version "9.0")
+	(generator_version "10.0")
 	(paper "A3")
 	(title_block
