File: z9-pdm/z9-pdm.kicad_sch (KiCad schematic)
At the start: 8 parts

Commit message: drc etc
Other:
- sheet MCU ports: added none; removed PC13
Changed lines of the file:
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@@
-		)
-	)
-	(label "VIPOWER_CS2"
-		(at 191.77 115.57 0)
-		(effects
-			(font
-				(size 1.27 1.27)
-			)
-			(justify left bottom)
 		)
 	)
@@
 			)
 		)
-		(pin "PC13" output
-			(at 191.77 115.57 0)
-			(effects
-				(font
-					(size 1.27 1.27)
-				)
-				(justify right)
-			)
-		)

Commit message: x
Parts:
- H1, H2, H3, H4, H5, H6, H7, H8: footprint MountingHole:MountingHole_4.3mm_M4_DIN965 -> dnt:MountingHole_4.3mm_M4_DIN965
Connections:
- no-connect marks 17 -> 12
Other:
- added sheet esp32-s3 (esp32-s3.kicad_sch)
- added sheet radio_433 (radio_433.kicad_sch)
- added sheet shared_ism330dhcx (../z9-shared/shared_ism330dhcx.kicad_sch)
- sheet MCU ports: added ESP_BOOT, ESP_EN, PC13, UART8_RX, UART8_TX; removed none
- note removed: "IIS3DHHCTR"

Commit message: x
Connections:
- no-connect marks 12 -> 0
Other:
- sheet MCU ports: added none; removed LCD_LED, LCD_ON, LCD_RESET, PC13, SENSOR_ON, SPI4_CS_1, SPI4_CS_2, SPI4_IRQ, SPI4_SCK, SPI4_SDI, SPI4_SDO, SYS_WKUP
Changed lines of the file:
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@@
 		(company "DNT")
-	)
-	(no_connect
-		(at 191.77 158.75)
-	)
-	(no_connect
-		(at 191.77 59.69)
-	)
-	(no_connect
-		(at 191.77 170.18)
-	)
-	(no_connect
-		(at 191.77 151.13)
-	)
-	(no_connect
-		(at 160.02 78.74)
-	)
-	(no_connect
-		(at 191.77 165.1)
-	)
-	(no_connect
-		(at 191.77 156.21)
-	)
-	(no_connect
-		(at 191.77 148.59)
-	)
-	(no_connect
-		(at 191.77 161.29)
-	)
-	(no_connect
-		(at 191.77 153.67)
-	)
-	(no_connect
-		(at 160.02 118.11)
-	)
-	(no_connect
-		(at 191.77 172.72)
 	)
 	(wire
@@
 			)
 		)
-		(pin "LCD_ON" output
-			(at 191.77 165.1 0)
-			(effects
-				(font
-					(size 1.27 1.27)
-				)
-				(justify right)
-			)
-		)
 		(pin "CAN1_RX" input
 			(at 191.77 180.34 0)
@@
 			)
 		)
-		(pin "LCD_LED" output
-			(at 191.77 170.18 0)
-			(effects
-				(font
-					(size 1.27 1.27)
-				)
-				(justify right)
-			)
-		)
-		(pin "LCD_RESET" output
-			(at 191.77 172.72 0)
-			(effects
-				(font
-					(size 1.27 1.27)
-				)
-				(justify right)
-			)
-		)
 		(pin "SPI2_IRQ2" input
 			(at 191.77 101.6 0)
@@
 			)
 		)
-		(pin "SPI4_CS_1" output
-			(at 191.77 153.67 0)
-			(effects
-				(font
-					(size 1.27 1.27)
-				)
-				(justify right)
-			)
-		)
-		(pin "SPI4_CS_2" output
-			(at 191.77 156.21 0)
-			(effects
-				(font
-					(size 1.27 1.27)
-				)
-				(justify right)
-			)
-		)
-		(pin "SPI4_IRQ" input
-			(at 191.77 158.75 0)
-			(effects
-				(font
-					(size 1.27 1.27)
-				)
-				(justify right)
-			)
-		)
 		(pin "SPI3_CS" output
 			(at 191.77 124.46 0)
@@
 			)
 		)
-		(pin "SYS_WKUP" input
-			(at 160.02 118.11 180)
-			(effects
-				(font
-					(size 1.27 1.27)
-				)
-				(justify left)
-			)
-		)
 		(pin "ADC1_IN6" input
 			(at 160.02 59.69 180)
@@
 			)
 		)
-		(pin "SENSOR_ON" output
-			(at 160.02 78.74 180)
-			(effects
-				(font
-					(size 1.27 1.27)
-				)
-				(justify left)
-			)
-		)
 		(pin "TIM3_CH1" output
 			(at 191.77 135.89 0)
@@
 			)
 		)
-		(pin "SPI4_SCK" output
-			(at 191.77 161.29 0)
-			(effects
-				(font
-					(size 1.27 1.27)
-				)
-				(justify right)
-			)
-		)
-		(pin "SPI4_SDI" input
-			(at 191.77 151.13 0)
-			(effects
-				(font
-					(size 1.27 1.27)
-				)
-				(justify right)
-			)
-		)
-		(pin "SPI4_SDO" output
-			(at 191.77 148.59 0)
-			(effects
-				(font
-					(size 1.27 1.27)
-				)
-				(justify right)
-			)
-		)
 		(pin "TIM1_CH3" output
 			(at 160.02 146.05 180)
@@
 			(effects
 				(font
-					(size 1.27 1.27)
-				)
-				(justify right)
-			)
-		)
-		(pin "PC13" output
-			(at 191.77 59.69 0)
-			(effects
-				(font

Commit message: x
Other:
- added sheet power_5v (untitled.kicad_sch)
Changed lines of the file:
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@@
+		)
+	)
+	(sheet
+		(at 222.25 231.14)
+		(size 49.53 39.37)
+		(exclude_from_sim no)
+		(in_bom yes)
+		(on_board yes)
+		(dnp no)
+		(fields_autoplaced yes)
+		(stroke
+			(width 0.1524)
+			(type solid)
+		)
+		(fill
+			(color 0 0 0 0.0000)
+		)
+		(property "Sheetname" "power_5v"
+			(at 222.25 230.4284 0)
+			(effects
+				(font
+					(size 1.27 1.27)
+				)
+				(justify left bottom)
+			)
+		)
+		(property "Sheetfile" "untitled.kicad_sch"
+			(at 222.25 271.0946 0)
+			(effects
+				(font
+					(size 1.27 1.27)
+				)
+				(justify left top)
+			)
+		)
+		(instances
+			(project "z9-pdm"
+				(path "/b643db5c-578e-4b48-aafc-cc4190db582a"
+					(page "24")
+				)
+			)
 		)
 	)

Commit message: new fuse and ideal diode
Other:
- sheet MCU ports: added PC13, TIM2_CH3; removed none
- sheet power ports: added 5VA_ENABLE; removed none

Commit message: post 5v lay references lost
Other:
- added sheet power_3.3V (power_3.3V.kicad_sch)
- added sheet power_5V_tba (power_5V_tba.kicad_sch)
Changed lines of the file:
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@@
+	)
+	(sheet
+		(at 233.045 202.565)
+		(size 59.69 19.05)
+		(exclude_from_sim no)
+		(in_bom yes)
+		(on_board yes)
+		(dnp no)
+		(fields_autoplaced yes)
+		(stroke
+			(width 0.1524)
+			(type solid)
+		)
+		(fill
+			(color 0 0 0 0.0000)
+		)
+		(property "Sheetname" "power_3.3V"
+			(at 233.045 201.8534 0)
+			(effects
+				(font
+					(size 1.27 1.27)
+				)
+				(justify left bottom)
+			)
+		)
+		(property "Sheetfile" "power_3.3V.kicad_sch"
+			(at 233.045 222.1996 0)
+			(effects
+				(font
+					(size 1.27 1.27)
+				)
+				(justify left top)
+			)
+		)
+		(instances
+			(project "z9-pdm"
+				(path "/b643db5c-578e-4b48-aafc-cc4190db582a"
+					(page "26")
+				)
+			)
+		)
 	)
 	(sheet
@@
 				)
 			)
+		)
+	)
+	(sheet
+		(at 233.045 171.45)
+		(size 59.69 17.78)
+		(exclude_from_sim no)
+		(in_bom yes)
+		(on_board yes)
+		(dnp no)
+		(fields_autoplaced yes)
+		(stroke
+			(width 0.1524)
+			(type solid)
+		)
+		(fill
+			(color 0 0 0 0.0000)
+		)
+		(property "Sheetname" "power_5V_tba"
+			(at 233.045 170.7384 0)
+			(effects
+				(font
+					(size 1.27 1.27)
+				)
+				(justify left bottom)
+			)
+		)
+		(property "Sheetfile" "power_5V_tba.kicad_sch"
+			(at 233.045 189.8146 0)
+			(effects
+				(font
+					(size 1.27 1.27)
+				)
+				(justify left top)
+			)
+		)
+		(instances
+			(project "z9-pdm"
+				(path "/b643db5c-578e-4b48-aafc-cc4190db582a"
+					(page "25")
+				)
+			)

Commit message: pre final pdm erc
Other:
- sheet MCU ports: added ADC1_IN9; removed none
- sheet connectors ports: added none; removed +5V_ISO
- sheet power ports: added IN_SENSE; removed 5VA_ENABLE
- sheet power_5V_tba ports: added 5VA_ENABLE; removed none
- sheet shared_can_isolated ports: added none; removed +5V_ISO
Changed lines of the file:
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@@
 	(wire
 		(pts
+			(xy 95.25 121.92) (xy 111.76 121.92)
+		)
+		(stroke
+			(width 0)
+			(type default)
+		)
+	)
+	(wire
+		(pts
 			(xy 304.8 69.85) (xy 312.42 69.85)
 		)
@@
 	)
 	(label "USB_OTG_FS_VBUS"
-		(at 93.98 215.9 0)
+		(at 93.98 177.165 0)
 		(effects
 			(font
@@
 	)
 	(label "ESP_BOOT"
-		(at 160.02 242.57 180)
-		(effects
-			(font
-				(size 1.27 1.27)
-			)
-			(justify right bottom)
-		)
-	)
-	(label "5VA_ENABLE"
-		(at 52.07 120.65 180)
+		(at 50.8 245.11 180)
 		(effects
 			(font
@@
 	)
 	(label "ESP_U0RXD"
-		(at 160.02 250.19 180)
+		(at 50.8 252.73 180)
 		(effects
 			(font
@@
 		)
 	)
+	(label "ADC1_IN9"
+		(at 111.76 121.92 0)
+		(effects
+			(font
+				(size 1.27 1.27)
+			)
+			(justify left bottom)
+		)
+	)
 	(label "VIPOWER_PWM"
 		(at 52.07 88.9 180)
@@
 	)
 	(label "ESP_EN"
-		(at 160.02 246.38 180)
+		(at 50.8 248.92 180)
 		(effects
 			(font
@@
 	)
 	(label "USB_OTG_FS_DP"
-		(at 93.98 200.66 0)
+		(at 93.98 161.925 0)
 		(effects
 			(font
@@
 	)
 	(label "ESP_U0TXD"
-		(at 160.02 254 180)
+		(at 50.8 256.54 180)
 		(effects
 			(font
@@
 		)
 	)
+	(label "5VA_ENABLE"
+		(at 233.045 177.8 180)
+		(effects
+			(font
+				(size 1.27 1.27)
+			)
+			(justify right bottom)
+		)
+	)
 	(label "ADC1_IN7"
 		(at 363.22 161.29 0)
@@
 	)
 	(label "USB_OTG_FS_DM"
-		(at 93.98 205.74 0)
+		(at 93.98 167.005 0)
 		(effects
 			(font
@@
 	)
 	(label "SPI2_IRQ"
-		(at 52.07 256.54 180)
+		(at 52.07 217.805 180)
 		(effects
 			(font
@@
 		)
 	)
+	(label "ADC1_IN9"
+		(at 160.02 83.82 180)
+		(effects
+			(font
+				(size 1.27 1.27)
+			)
+			(justify right bottom)
+		)
+	)
 	(label "SENSE_5"
 		(at 312.42 157.48 180)
@@
 		)
 	)
-	(label "+5V_ISO"
-		(at 52.07 38.1 180)
-		(effects
-			(font
-				(size 1.27 1.27)
-			)
-			(justify right bottom)
-		)
-	)
 	(label "SPI2_SDO"
-		(at 52.07 242.57 180)
+		(at 52.07 203.835 180)
 		(effects
 			(font
@@
 	)
 	(label "BUZZER"
-		(at 52.07 179.07 180)
+		(at 52.07 140.335 180)
 		(effects
 			(font
@@
 	)
 	(label "SPI2_IRQ2"
-		(at 52.07 260.35 180)
+		(at 52.07 221.615 180)
 		(effects
 			(font
@@
 		)
 	)
-	(label "+5V_ISO"
-		(at 312.42 92.71 180)
-		(effects
-			(font
-				(size 1.27 1.27)
-			)
-			(justify right bottom)
-		)
-	)
 	(label "ADC1_IN3"
 		(at 363.22 153.67 0)
@@
 	)
 	(label "SPI2_CS"
-		(at 52.07 234.95 180)
+		(at 52.07 196.215 180)
 		(effects
 			(font
@@
 	)
 	(label "SPI2_SDI"
-		(at 52.07 246.38 180)
+		(at 52.07 207.645 180)
 		(effects
 			(font
@@
 	)
 	(label "SPI2_SCK"
-		(at 52.07 238.76 180)
+		(at 52.07 200.025 180)
 		(effects
 			(font
@@
 			)
 		)
+		(pin "ADC1_IN9" input
+			(at 160.02 83.82 180)
+			(effects
+				(font
+					(size 1.27 1.27)
+				)
+				(justify left)
+			)
+		)
 		(instances
 			(project "z9-pdm"
@@
 	)
 	(sheet
-		(at 160.02 231.14)
-		(size 31.75 39.37)
+		(at 50.8 233.68)
+		(size 44.45 39.37)
 		(exclude_from_sim no)
 		(in_bom yes)
@@
 		)
 		(property "Sheetname" "esp32-s3"
-			(at 160.02 230.4284 0)
+			(at 50.8 232.9684 0)
 			(effects
 				(font
@@
 		)
 		(property "Sheetfile" "esp32-s3.kicad_sch"
-			(at 160.02 271.0946 0)
+			(at 50.8 273.6346 0)
 			(effects
 				(font
@@
 		)
 		(pin "ESP_BOOT" input
-			(at 160.02 242.57 180)
+			(at 50.8 245.11 180)
 			(effects
 				(font
@@
 		)
 		(pin "ESP_EN" input
-			(at 160.02 246.38 180)
+			(at 50.8 248.92 180)
 			(effects
 				(font
@@
 		)
 		(pin "ESP_U0RXD" input
-			(at 160.02 250.19 180)
+			(at 50.8 252.73 180)
 			(effects
 				(font
@@
 		)
 		(pin "ESP_U0TXD" output
-			(at 160.02 254 180)
+			(at 50.8 256.54 180)
 			(effects
 				(font
@@
 			)
 		)
-		(pin "+5V_ISO" input
-			(at 52.07 38.1 180)
-			(effects
-				(font
-					(size 1.27 1.27)
-				)
-				(justify left)
-			)
-		)
 		(pin "CAN_H" bidirectional
 			(at 95.25 26.67 0)
@@
 			)
 		)
+		(pin "5VA_ENABLE" input
+			(at 233.045 177.8 180)
+			(effects
+				(font
+					(size 1.27 1.27)
+				)
+				(justify left)
+			)
+		)
 		(instances
 			(project "z9-pdm"
@@
 			)
 		)
-		(pin "+5V_ISO" output
-			(at 312.42 92.71 180)
-			(effects
-				(font
-					(size 1.27 1.27)
-				)
-				(justify left)
-			)
-		)
 		(pin "GND_ISO" bidirectional
 			(at 312.42 88.9 180)
@@
 	)
 	(sheet
-		(at 52.07 231.14)
+		(at 52.07 192.405)
 		(size 41.91 31.75)
 		(exclude_from_sim no)
@@
 		)
 		(property "Sheetname" "shared_ism330dhcx"
-			(at 52.07 230.4284 0)
+			(at 52.07 191.6934 0)
 			(effects
 				(font
@@
 		)
 		(property "Sheetfile" "../z9-shared/shared_ism330dhcx.kicad_sch"
-			(at 52.07 263.4746 0)
+			(at 52.07 224.7396 0)
 			(effects
 				(font
@@
 		)
 		(pin "ISM_CS" input
-			(at 52.07 234.95 180)
+			(at 52.07 196.215 180)
 			(effects
 				(font
@@
 		)
 		(pin "ISM_INT1" input
-			(at 52.07 256.54 180)
+			(at 52.07 217.805 180)
 			(effects
 				(font
@@
 		)
 		(pin "ISM_INT2" input
-			(at 52.07 260.35 180)
+			(at 52.07 221.615 180)
 			(effects
 				(font
@@
 		)
 		(pin "ISM_SCK" input
-			(at 52.07 238.76 180)
+			(at 52.07 200.025 180)
 			(effects
 				(font
@@
 		)
 		(pin "ISM_SDI" input
-			(at 52.07 242.57 180)
+			(at 52.07 203.835 180)
 			(effects
 				(font
@@
 		)
 		(pin "ISM_SDO" input
-			(at 52.07 246.38 180)
+			(at 52.07 207.645 180)
 			(effects
 				(font
@@
 	)
 	(sheet
-		(at 52.07 196.85)
+		(at 52.07 158.115)
 		(size 41.91 24.13)
 		(exclude_from_sim no)
@@
 		)
 		(property "Sheetname" "shared_usbc"
-			(at 52.07 196.1384 0)
+			(at 52.07 157.4034 0)
 			(effects
 				(font
@@
 		)
 		(property "Sheetfile" "../z9-shared/shared_usbc.kicad_sch"
-			(at 52.07 221.5646 0)
+			(at 52.07 182.8296 0)
 			(effects
 				(font
@@
 		)
 		(pin "USB_OTG_FS_DP" bidirectional
-			(at 93.98 200.66 0)
+			(at 93.98 161.925 0)
 			(effects
 				(font
@@
 		)
 		(pin "USB_OTG_FS_DM" bidirectional
-			(at 93.98 205.74 0)
+			(at 93.98 167.005 0)
 			(effects
 				(font
@@
 		)
 		(pin "USB_OTG_FS_VBUS" output
-			(at 93.98 215.9 0)
+			(at 93.98 177.165 0)
 			(effects
 				(font
@@
 	)
 	(sheet
-		(at 52.07 173.99)
+		(at 52.07 135.255)
 		(size 41.91 11.43)
 		(exclude_from_sim no)
@@
 		)
 		(property "Sheetname" "shared_buzzer_2"
-			(at 52.07 173.2784 0)
+			(at 52.07 134.5434 0)
 			(effects
 				(font
@@
 		)
 		(property "Sheetfile" "../z9-shared/shared_buzzer.kicad_sch"
-			(at 52.07 186.0046 0)
+			(at 52.07 147.2696 0)
 			(effects
 				(font
@@
 		)
 		(pin "BUZZER" input
-			(at 52.07 179.07 180)
+			(at 52.07 140.335 180)
 			(effects
 				(font
@@
 	(sheet
 		(at 52.07 114.3)
-		(size 40.64 44.45)
+		(size 43.18 12.7)
 		(exclude_from_sim no)
 		(in_bom yes)
@@
 		)
 		(property "Sheetfile" "power.kicad_sch"
-			(at 52.07 159.3346 0)
+			(at 52.07 127.5846 0)
 			(effects
 				(font
@@
 			)
 		)
-		(pin "5VA_ENABLE" input
-			(at 52.07 120.65 180)
+		(pin "IN_SENSE" output
+			(at 95.25 121.92 0)
 			(effects
 				(font
 					(size 1.27 1.27)
 				)
-				(justify left)
+				(justify right)
 			)
 		)

Commit message: x
Parts:
- renumbered H8 to H2, H7 to H3, H6 to H4, H1 to H6, H2 to H7, H3 to H8, H4 to H9
