File: z9-pdm/analogue_input_stage.kicad_sch (KiCad schematic)
At the start: 6 parts

Commit message: x
Parts:
- D14: value PESD24VF1BLYL -> ~; footprint PCM_Diode_SMD_AKL:D_SOD-323_TVS -> PCM_Diode_SMD_AKL:D_SOD-882_DFN1006-2_TVS; symbol PCM_Diode_TVS_AKL:PESD24VL1BA -> dnt_global:PESD30VF1BLYL; LCSC C2443373 -> (none)
Changed lines of the file:
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@@
 		)
 		(instances
-			(project ""
+			(project "z9-pdm"
 				(path "/b643db5c-578e-4b48-aafc-cc4190db582a/4bf3a54e-2413-4742-bb3c-6ced251716e8/16936357-08be-4dfb-9389-5ff776d9b4b6"
 					(reference "R45")
@@
 		)
 		(instances
-			(project "z9-pdm-pcb"
+			(project "z9-pdm"
 				(path "/b643db5c-578e-4b48-aafc-cc4190db582a/4bf3a54e-2413-4742-bb3c-6ced251716e8/16936357-08be-4dfb-9389-5ff776d9b4b6"
 					(reference "#PWR093")
@@
 	)
 	(symbol
-		(lib_id "PCM_Diode_TVS_AKL:PESD24VL1BA")
+		(lib_id "dnt_global:PESD30VF1BLYL")
 		(at 156.21 77.47 90)
 		(unit 1)
@@
 		(fields_autoplaced yes)
 		(property "Reference" "D14"
-			(at 158.75 76.1999 90)
+			(at 158.75 77.4699 90)
 			(effects
 				(font
@@
 			)
 		)
-		(property "Value" "PESD24VF1BLYL"
+		(property "Value" "~"
 			(at 158.75 78.7399 90)
 			(effects
@@
 			)
 		)
-		(property "Footprint" "PCM_Diode_SMD_AKL:D_SOD-323_TVS"
+		(property "Footprint" "PCM_Diode_SMD_AKL:D_SOD-882_DFN1006-2_TVS"
 			(at 156.21 77.47 0)
 			(effects
@@
 			)
 		)
-		(property "Datasheet" "https://www.tme.eu/Document/952767affdffba4b305eacda1aae6cd9/PESD24VL1BA-DTE.pdf"
+		(property "Datasheet" "https://www.tme.eu/Document/6d36879fb2dd3d2490c58510ca5e3957/PESD5V0S1BB-DTE.pdf"
 			(at 156.21 77.47 0)
 			(effects
@@
 			)
 		)
-		(property "Description" "SOD-323 Bidirectional TVS Diode, 24V, 200W, Alternate KiCAD Library"
-			(at 156.21 77.47 0)
-			(effects
-				(font
-					(size 1.27 1.27)
-				)
-				(hide yes)
-			)
-		)
-		(property "LCSC" "C2443373"
+		(property "Description" "SOD-882 Bidirectional TVS Diode, 5V, 130W, Alternate KiCAD Library"
 			(at 156.21 77.47 0)
 			(effects
@@
 		)
 		(instances
-			(project "z9-pdm-pcb"
+			(project "z9-pdm"
 				(path "/b643db5c-578e-4b48-aafc-cc4190db582a/4bf3a54e-2413-4742-bb3c-6ced251716e8/16936357-08be-4dfb-9389-5ff776d9b4b6"
 					(reference "R47")
@@
 		)
 		(instances
-			(project "z9-pdm-pcb"
+			(project "z9-pdm"
 				(path "/b643db5c-578e-4b48-aafc-cc4190db582a/4bf3a54e-2413-4742-bb3c-6ced251716e8/16936357-08be-4dfb-9389-5ff776d9b4b6"
 					(reference "C43")
@@
 		)
 		(instances
-			(project ""
+			(project "z9-pdm"
 				(path "/b643db5c-578e-4b48-aafc-cc4190db582a/4bf3a54e-2413-4742-bb3c-6ced251716e8/16936357-08be-4dfb-9389-5ff776d9b4b6"
 					(reference "D19")
@@
 		)
 		(instances
-			(project "z9-pdm-pcb"
+			(project "z9-pdm"
 				(path "/b643db5c-578e-4b48-aafc-cc4190db582a/4bf3a54e-2413-4742-bb3c-6ced251716e8/16936357-08be-4dfb-9389-5ff776d9b4b6"
 					(reference "R46")
