File: z9-pdm/analogue_input_stage.kicad_sch (KiCad schematic)
At the start: 7 parts

Commit message: pre replicate analogue chans
Parts:
- removed C29: 1nF, PCM_JLCPCB:C_0603, symbol PCM_JLCPCB-Capacitors:0603,1nF
- removed D18: SMBJ24CA, PCM_Diode_SMD_AKL:D_SMB_TVS, symbol PCM_Diode_TVS_AKL:SMBJ24CA
- removed F4: Fuse_16V_500mA_100A_1A_150mΩ_0805_PTC_Resettable_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, Fuse:Fuse_0805_2012Metric, symbol dnt_global:Fuse_16V_500mA_100A_1A_150mΩ_0805_PTC_Resettable_Fuses_ROHS
- removed R25: 100Ω, PCM_JLCPCB:R_0603, symbol PCM_JLCPCB-Resistors:0603,100Ω
- added D5001: PESD24VF1BLYL, PCM_Diode_SMD_AKL:D_SOD-323_TVS, symbol PCM_Diode_TVS_AKL:PESD24VL1BA
- added D5002: BAT54S, Package_TO_SOT_SMD:SOT-23, symbol Diode:BAT54S
- added R5001: 1kΩ, PCM_JLCPCB:R_0805, symbol PCM_JLCPCB-Resistors:0805,1kΩ
- renumbered C31 to C5001, R26 to R5002, R27 to R5003
Connections:
- net AD_IN: now also D5002.3 (COM)
- net GND: now also D5001.1 (K), D5002.1 (A)
- net SENSE: now also R5001.1
- net at R5002.2: now also D5001.2 (A), R5001.2
- new net 3V3_VOLT: D5002.2 (K)
Other:
- moved on the sheet: R5002, R5003

Commit message: x
Parts:
- D14: renamed from D5001; LCSC (none) -> C2443373
- D15: renamed from D5002; symbol Diode:BAT54S -> dnt_global:BAT54S; LCSC (none) -> C19726
- renumbered C5001 to C41, R5001 to R39, R5002 to R40, R5003 to R41

Commit message: passes sch drc
Changed lines of the file:
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@@
 		)
 		(property "Value" "GND"
-			(at 166.37 109.2199 0)
+			(at 163.83 113.03 0)
 			(effects
 				(font
 					(size 1.27 1.27)
 				)
-				(justify left)
 			)
 		)

Commit message: jlc
Parts:
- R41: footprint PCM_JLCPCB:R_0603 -> dnt:R_0402_1005Metric; symbol PCM_JLCPCB-Resistors:0603,10kΩ -> dnt_global:0402,10kΩ; LCSC C25804 -> C25744; Overload Voltage (Max) 75V -> 50V; Part 0603WAF1002T5E -> 0402WGF1002TCE; Power(Watts) 100mW -> 62.5mW; Stock 51181774 -> 24372091
Changed lines of the file:
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@@
 	)
 	(symbol
-		(lib_id "PCM_JLCPCB-Resistors:0603,10kΩ")
+		(lib_id "dnt_global:0402,10kΩ")
 		(at 180.34 74.93 0)
 		(mirror x)
@@
 			)
 		)
-		(property "Footprint" "PCM_JLCPCB:R_0603"
+		(property "Footprint" "dnt:R_0402_1005Metric"
 			(at 178.562 74.93 90)
 			(effects
@@
 			)
 		)
-		(property "Datasheet" "https://www.lcsc.com/datasheet/lcsc_datasheet_2206010045_UNI-ROYAL-Uniroyal-Elec-0603WAF1002T5E_C25804.pdf"
+		(property "Datasheet" "https://www.lcsc.com/datasheet/lcsc_datasheet_2411221126_UNI-ROYAL-Uniroyal-Elec-0402WGF1002TCE_C25744.pdf"
 			(at 180.34 74.93 0)
 			(effects
@@
 			)
 		)
-		(property "Description" "100mW Thick Film Resistors 75V ±100ppm/°C ±1% 10kΩ 0603 Chip Resistor - Surface Mount ROHS"
+		(property "Description" "62.5mW Thick Film Resistors 50V ±100ppm/°C ±1% 10kΩ 0402 Chip Resistor - Surface Mount ROHS"
 			(at 180.34 74.93 0)
 			(effects
@@
 			)
 		)
-		(property "LCSC" "C25804"
+		(property "LCSC" "C25744"
 			(at 180.34 74.93 0)
 			(effects
@@
 			)
 		)
-		(property "Stock" "51181774"
+		(property "Stock" "24372091"
 			(at 180.34 74.93 0)
 			(effects
@@
 			)
 		)
-		(property "Part" "0603WAF1002T5E"
+		(property "Part" "0402WGF1002TCE"
 			(at 180.34 74.93 0)
 			(effects
@@
 			)
 		)
-		(property "Power(Watts)" "100mW"
+		(property "Power(Watts)" "62.5mW"
 			(at 180.34 74.93 0)
 			(effects
@@
 			)
 		)
-		(property "Overload Voltage (Max)" "75V"
+		(property "Overload Voltage (Max)" "50V"
 			(at 180.34 74.93 0)
 			(effects

Commit message: jlc
Parts:
- D14: footprint PCM_Diode_SMD_AKL:D_SOD-323_TVS -> PCM_Diode_SMD_AKL:D_SOD-882_DFN1006-2_TVS; symbol PCM_Diode_TVS_AKL:PESD24VL1BA -> dnt_global:PESD30VF1BLYL; LCSC C2443373 -> (none)
Changed lines of the file:
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@@
 		)
 		(instances
-			(project ""
+			(project "z9-pdm"
 				(path "/b643db5c-578e-4b48-aafc-cc4190db582a/4bf3a54e-2413-4742-bb3c-6ced251716e8/16936357-08be-4dfb-9389-5ff776d9b4b6"
 					(reference "R45")
@@
 		)
 		(instances
-			(project "z9-pdm-pcb"
+			(project "z9-pdm"
 				(path "/b643db5c-578e-4b48-aafc-cc4190db582a/4bf3a54e-2413-4742-bb3c-6ced251716e8/16936357-08be-4dfb-9389-5ff776d9b4b6"
 					(reference "#PWR093")
@@
 	)
 	(symbol
-		(lib_id "PCM_Diode_TVS_AKL:PESD24VL1BA")
+		(lib_id "dnt_global:PESD30VF1BLYL")
 		(at 156.21 77.47 90)
 		(unit 1)
@@
 			)
 		)
-		(property "Footprint" "PCM_Diode_SMD_AKL:D_SOD-323_TVS"
+		(property "Footprint" "PCM_Diode_SMD_AKL:D_SOD-882_DFN1006-2_TVS"
 			(at 156.21 77.47 0)
 			(effects
@@
 			)
 		)
-		(property "Datasheet" "https://www.tme.eu/Document/952767affdffba4b305eacda1aae6cd9/PESD24VL1BA-DTE.pdf"
+		(property "Datasheet" "https://www.tme.eu/Document/6d36879fb2dd3d2490c58510ca5e3957/PESD5V0S1BB-DTE.pdf"
 			(at 156.21 77.47 0)
 			(effects
@@
 			)
 		)
-		(property "Description" "SOD-323 Bidirectional TVS Diode, 24V, 200W, Alternate KiCAD Library"
-			(at 156.21 77.47 0)
-			(effects
-				(font
-					(size 1.27 1.27)
-				)
-				(hide yes)
-			)
-		)
-		(property "LCSC" "C2443373"
+		(property "Description" "SOD-882 Bidirectional TVS Diode, 5V, 130W, Alternate KiCAD Library"
 			(at 156.21 77.47 0)
 			(effects
@@
 		)
 		(instances
-			(project "z9-pdm-pcb"
+			(project "z9-pdm"
 				(path "/b643db5c-578e-4b48-aafc-cc4190db582a/4bf3a54e-2413-4742-bb3c-6ced251716e8/16936357-08be-4dfb-9389-5ff776d9b4b6"
 					(reference "R47")
@@
 		)
 		(instances
-			(project "z9-pdm-pcb"
+			(project "z9-pdm"
 				(path "/b643db5c-578e-4b48-aafc-cc4190db582a/4bf3a54e-2413-4742-bb3c-6ced251716e8/16936357-08be-4dfb-9389-5ff776d9b4b6"
 					(reference "C43")
@@
 		)
 		(instances
-			(project ""
+			(project "z9-pdm"
 				(path "/b643db5c-578e-4b48-aafc-cc4190db582a/4bf3a54e-2413-4742-bb3c-6ced251716e8/16936357-08be-4dfb-9389-5ff776d9b4b6"
 					(reference "D19")
@@
 		)
 		(instances
-			(project "z9-pdm-pcb"
+			(project "z9-pdm"
 				(path "/b643db5c-578e-4b48-aafc-cc4190db582a/4bf3a54e-2413-4742-bb3c-6ced251716e8/16936357-08be-4dfb-9389-5ff776d9b4b6"
 					(reference "R46")
