File: z9-pdm/connectors.kicad_sch (KiCad schematic)
At the start: 11 parts, among them J10 Wago 12 pin 1 level 3.5mm 260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, J11 TE_DT15-12PC-B016 -Conn_01x12, J12 Wago 12 pin 1 level 3.5mm 260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, J13 TE_DT15-12PC-B016 -Conn_01x12, J14 Wago 12 pin 1 level 3.5mm 260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, J15 TE_DT15-12PC-B016 -Conn_01x12, J5 JST GH, J6 Wago 12 pin 1 level 3.5mm 260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, J7 TE_DT15-12PC-B016 -Conn_01x12, J8 RedCubeTerminal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

Commit message: jlc
Parts:
- J5: LCSC C189892 -> C160392
Changed lines of the file:
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@@
 			)
 		)
-		(property "LCSC" "C189892"
+		(property "LCSC" "C160392"
 			(at 67.31 177.038 0)
 			(effects

Commit message: x
Parts:
- J5: value JST GH -> BM06B-GHS-GB-TBT(LF)(SN)(N); LCSC C160392 -> C17467557; now not fitted; now left out of the parts list
Changed lines of the file:
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@@
 		)
 		(instances
-			(project "z9-pdm-pcb"
+			(project "z9-pdm"
 				(path "/b643db5c-578e-4b48-aafc-cc4190db582a/651fe70f-48a4-454d-84e2-56b28624b7c9"
 					(reference "J14")
@@
 		(unit 1)
 		(exclude_from_sim no)
-		(in_bom yes)
-		(on_board yes)
-		(dnp no)
+		(in_bom no)
+		(on_board yes)
+		(dnp yes)
 		(fields_autoplaced yes)
 		(property "Reference" "J5"
@@
 			)
 		)
-		(property "Value" "JST  GH"
+		(property "Value" "BM06B-GHS-GB-TBT(LF)(SN)(N)"
 			(at 67.31 157.48 0)
 			(effects
@@
 			)
 		)
-		(property "Datasheet" "https://wmsc.lcsc.com/wmsc/upload/file/pdf/v2/lcsc/2304140030_JST-BM06B-GHS-TBT-LF-SN_C189892.pdf"
+		(property "Datasheet" ""
 			(at 67.31 179.07 0)
 			(effects
@@
 			)
 		)
-		(property "Description" "JST Connector  6 pins"
+		(property "Description" "-25℃~+85℃ 1 1.25mm 10.75mm 1A 1x6P 4.05mm 4.32mm 50V 6 6P Auxiliary Solder Pin GH Gold PA9T Phosphor Bronze Surface Mount,Vertical UL94V-0 White SMD,P=1.25mm Wire To Board Connector ROHS"
 			(at 68.072 150.368 0)
 			(effects
@@
 			)
 		)
-		(property "LCSC" "C160392"
+		(property "LCSC" "C17467557"
 			(at 67.31 177.038 0)
 			(effects
@@
 		)
 		(instances
-			(project "z9-pdm-pcb"
+			(project "z9-pdm"
 				(path "/b643db5c-578e-4b48-aafc-cc4190db582a/651fe70f-48a4-454d-84e2-56b28624b7c9"
 					(reference "J5")
@@
 		)
 		(instances
-			(project "z9-pdm-pcb"
+			(project "z9-pdm"
 				(path "/b643db5c-578e-4b48-aafc-cc4190db582a/651fe70f-48a4-454d-84e2-56b28624b7c9"
 					(reference "J9")
@@
 		)
 		(instances
-			(project "z9-pdm-pcb"
+			(project "z9-pdm"
 				(path "/b643db5c-578e-4b48-aafc-cc4190db582a/651fe70f-48a4-454d-84e2-56b28624b7c9"
 					(reference "J7")
@@
 		)
 		(instances
-			(project ""
+			(project "z9-pdm"
 				(path "/b643db5c-578e-4b48-aafc-cc4190db582a/651fe70f-48a4-454d-84e2-56b28624b7c9"
 					(reference "#PWR046")
@@
 		)
 		(instances
-			(project "z9-pdm-pcb"
+			(project "z9-pdm"
 				(path "/b643db5c-578e-4b48-aafc-cc4190db582a/651fe70f-48a4-454d-84e2-56b28624b7c9"
 					(reference "J10")
@@
 		)
 		(instances
-			(project "z9-pdm-pcb"
+			(project "z9-pdm"
 				(path "/b643db5c-578e-4b48-aafc-cc4190db582a/651fe70f-48a4-454d-84e2-56b28624b7c9"
 					(reference "#PWR052")
@@
 		)
 		(instances
-			(project "z9-pdm-pcb"
+			(project "z9-pdm"
 				(path "/b643db5c-578e-4b48-aafc-cc4190db582a/651fe70f-48a4-454d-84e2-56b28624b7c9"
 					(reference "J11")
@@
 		)
 		(instances
-			(project "z9-pdm-pcb"
+			(project "z9-pdm"
 				(path "/b643db5c-578e-4b48-aafc-cc4190db582a/651fe70f-48a4-454d-84e2-56b28624b7c9"
 					(reference "J13")
@@
 		)
 		(instances
-			(project "z9-pdm-pcb"
+			(project "z9-pdm"
 				(path "/b643db5c-578e-4b48-aafc-cc4190db582a/651fe70f-48a4-454d-84e2-56b28624b7c9"
 					(reference "#PWR051")
@@
 		)
 		(instances
-			(project "z9-pdm-pcb"
+			(project "z9-pdm"
 				(path "/b643db5c-578e-4b48-aafc-cc4190db582a/651fe70f-48a4-454d-84e2-56b28624b7c9"
 					(reference "J15")
@@
 		)
 		(instances
-			(project "z9-pdm-pcb"
+			(project "z9-pdm"
 				(path "/b643db5c-578e-4b48-aafc-cc4190db582a/651fe70f-48a4-454d-84e2-56b28624b7c9"
 					(reference "J8")
@@
 		)
 		(instances
-			(project "z9-pdm-pcb"
+			(project "z9-pdm"
 				(path "/b643db5c-578e-4b48-aafc-cc4190db582a/651fe70f-48a4-454d-84e2-56b28624b7c9"
 					(reference "#PWR047")
@@
 		)
 		(instances
-			(project "z9-pdm-pcb"
+			(project "z9-pdm"
 				(path "/b643db5c-578e-4b48-aafc-cc4190db582a/651fe70f-48a4-454d-84e2-56b28624b7c9"
 					(reference "J12")
@@
 		)
 		(instances
-			(project "z9-pdm-pcb"
+			(project "z9-pdm"
 				(path "/b643db5c-578e-4b48-aafc-cc4190db582a/651fe70f-48a4-454d-84e2-56b28624b7c9"
 					(reference "#PWR050")
@@
 		)
 		(instances
-			(project "z9-pdm-pcb"
+			(project "z9-pdm"
 				(path "/b643db5c-578e-4b48-aafc-cc4190db582a/651fe70f-48a4-454d-84e2-56b28624b7c9"
 					(reference "J6")
@@
 		)
 		(instances
-			(project "z9-pdm-pcb"
+			(project "z9-pdm"
 				(path "/b643db5c-578e-4b48-aafc-cc4190db582a/651fe70f-48a4-454d-84e2-56b28624b7c9"
 					(reference "#PWR049")
