File: z9-pdm/power_3.3V.kicad_sch (KiCad schematic)
At the start: 11 parts, among them U1 TLV76733DRVx, U2 TLV76733DRVx

Commit message: x
Parts:
- TP4: renamed from TP2; value PE0 -> +3.3V; now in the parts list
- U11: renamed from U2; symbol Regulator_Linear:TLV76733DRVx -> dnt_global:TLV76733DRVx; LCSC (none) -> C2848334
- U12: renamed from U1; symbol Regulator_Linear:TLV76733DRVx -> dnt_global:TLV76733DRVx; LCSC (none) -> C2848334
- renumbered C3 to C37, C2 to C38, C5 to C39, C4 to C40, D9 to D13, F4 to F7, F3 to F8, R4 to R38

Commit message: passes sch drc
Changed lines of the file:
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@@
 		)
 		(property "Value" "Fuse_16V_500mA_100A_1A_150mΩ_PTC"
-			(at 171.45 59.69 90)
+			(at 161.544 54.61 90)
 			(effects
 				(font
@@
 					(size 1.27 1.27)
 				)
+				(hide yes)
 			)
 		)
@@
 					(size 1.27 1.27)
 				)
+				(hide yes)
 			)
 		)
@@
 		)
 		(property "Value" "+5V"
-			(at 123.19 62.2299 0)
-			(effects
-				(font
-					(size 1.27 1.27)
-				)
-				(justify left)
+			(at 120.65 58.42 0)
+			(effects
+				(font
+					(size 1.27 1.27)
+				)
 			)
 		)
@@
 		)
 		(property "Value" "+3.3VA"
-			(at 175.26 109.2199 0)
-			(effects
-				(font
-					(size 1.27 1.27)
-				)
-				(justify left)
+			(at 172.72 105.41 0)
+			(effects
+				(font
+					(size 1.27 1.27)
+				)
 			)
 		)
@@
 				)
 				(justify left)
+				(hide yes)
 			)
 		)
@@
 		)
 		(property "Value" "+5VA"
-			(at 124.46 113.0299 0)
-			(effects
-				(font
-					(size 1.27 1.27)
-				)
-				(justify left)
+			(at 121.92 109.22 0)
+			(effects
+				(font
+					(size 1.27 1.27)
+				)
 			)
 		)
@@
 		)
 		(property "Value" "Fuse_16V_500mA_100A_1A_150mΩ_PTC"
-			(at 165.1 118.618 90)
+			(at 159.512 104.648 90)
 			(effects
 				(font
@@
 				)
 				(justify left)
-			)
-		)
+				(hide yes)
+			)
+		)
