File: z9-pdm/power_5V_tba.kicad_sch (KiCad schematic)
At the start: 28 parts, among them U6 LMR14206, U7 LMR14206

Commit message: pre final pdm erc
Changed lines of the file:
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@@
-	(wire
-		(pts
-			(xy 217.17 58.42) (xy 217.17 59.69)
-		)
-		(stroke
-			(width 0)
-			(type default)
-		)
-	)
 	(wire
 		(pts

Commit message: x
Parts:
- TP2: renamed from TP3; value PE0 -> +5V; now in the parts list
- TP3: renamed from TP5; now in the parts list
- renumbered C6 to C31, C18 to C32, C7 to C33, C19 to C34, C10 to C35, C21 to C36, D21 to D10, D19 to D11, D22 to D12, D3 to D7, D12 to D9, F5 to F3, F7 to F4, F6 to F5, F8 to F6, R8 to R32, R9 to R33, R16 to R34, R17 to R35, R10 to R36, R18 to R37, U7 to U10, U6 to U9

Commit message: passes sch drc
Parts:
- U10, U9: symbol Regulator_Switching:LMR14206 -> dnt_global:LMR14206; LCSC (none) -> C48239
Changed lines of the file:
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@@
 		)
 		(property "Value" "+5V"
-			(at 210.82 48.2599 0)
+			(at 208.28 44.45 0)
 			(effects
 				(font
 					(size 1.27 1.27)
 				)
-				(justify left)
 			)
 		)
@@
 		)
 		(property "Value" "+12V_VIPOWER"
-			(at 92.71 45.7199 0)
+			(at 90.17 41.91 0)
 			(effects
 				(font
 					(size 1.27 1.27)
 				)
-				(justify left)
 			)
 		)
@@
 		)
 		(property "Value" "PWR_FLAG"
-			(at 222.25 111.7599 0)
+			(at 219.71 107.95 0)
 			(effects
 				(font
 					(size 1.27 1.27)
 				)
-				(justify left)
 			)
 		)
@@
 		)
 		(property "Value" "PWR_FLAG"
-			(at 119.38 111.7599 0)
+			(at 116.84 107.95 0)
 			(effects
 				(font
 					(size 1.27 1.27)
 				)
-				(justify left)
 			)
 		)
@@
 	)
 	(symbol
-		(lib_id "Regulator_Switching:LMR14206")
+		(lib_id "dnt_global:LMR14206")
 		(at 140.97 121.92 0)
 		(unit 1)
@@
 			)
 		)
+		(property "LCSC" "C48239"
+			(at 140.97 121.92 0)
+			(effects
+				(font
+					(size 1.27 1.27)
+				)
+				(hide yes)
+			)
+		)
 		(pin "4"
 		)
@@
 		)
 		(property "Value" "PWR_FLAG"
-			(at 219.71 49.5299 0)
+			(at 217.17 45.72 0)
 			(effects
 				(font
 					(size 1.27 1.27)
 				)
-				(justify left)
 			)
 		)
@@
 		)
 		(property "Value" "PWR_FLAG"
-			(at 104.14 49.5299 0)
+			(at 101.6 45.72 0)
 			(effects
 				(font
 					(size 1.27 1.27)
 				)
-				(justify left)
 			)
 		)
@@
 		)
 		(property "Value" "+12V_VIPOWER"
-			(at 97.79 111.7599 0)
+			(at 95.25 107.95 0)
 			(effects
 				(font
 					(size 1.27 1.27)
 				)
-				(justify left)
 			)
 		)
@@
 	)
 	(symbol
-		(lib_id "Regulator_Switching:LMR14206")
+		(lib_id "dnt_global:LMR14206")
 		(at 138.43 59.69 0)
 		(unit 1)
@@
 			)
 		)
+		(property "LCSC" "C48239"
+			(at 138.43 59.69 0)
+			(effects
+				(font
+					(size 1.27 1.27)
+				)
+				(hide yes)
+			)
+		)
 		(pin "4"
 		)
@@
 		)
 		(property "Value" "+5VA"
-			(at 213.36 110.4899 0)
+			(at 210.82 106.68 0)
 			(effects
 				(font
 					(size 1.27 1.27)
 				)
-				(justify left)
 			)
 		)
