File: z9-pdm/radio_433.kicad_sch (KiCad schematic)
At the start: 10 parts, among them U2301 RXB6_radio_receiver

Commit message: pre kc update
Connections:
- net GND: now also U2301.2 (GND), U2301.3 (GND)
Changed lines of the file:
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@@
+	)
+	(junction
+		(at 177.8 87.63)
+		(diameter 0)
+		(color 0 0 0 0)
 	)
 	(junction
@@
 	)
 	(junction
-		(at 153.67 128.27)
+		(at 119.38 125.73)
 		(diameter 0)
 		(color 0 0 0 0)
@@
 	(wire
 		(pts
+			(xy 177.8 87.63) (xy 189.23 87.63)
+		)
+		(stroke
+			(width 0)
+			(type default)
+		)
+	)
+	(wire
+		(pts
+			(xy 119.38 123.19) (xy 119.38 125.73)
+		)
+		(stroke
+			(width 0)
+			(type default)
+		)
+	)
+	(wire
+		(pts
 			(xy 153.67 123.19) (xy 184.15 123.19)
 		)
@@
 	(wire
 		(pts
-			(xy 167.64 87.63) (xy 189.23 87.63)
-		)
-		(stroke
-			(width 0)
-			(type default)
-		)
-	)
-	(wire
-		(pts
-			(xy 152.4 128.27) (xy 153.67 128.27)
+			(xy 167.64 87.63) (xy 177.8 87.63)
 		)
 		(stroke
@@
 	(wire
 		(pts
+			(xy 119.38 125.73) (xy 119.38 137.16)
+		)
+		(stroke
+			(width 0)
+			(type default)
+		)
+	)
+	(wire
+		(pts
 			(xy 201.93 87.63) (xy 189.23 87.63)
 		)
@@
 	(wire
 		(pts
+			(xy 119.38 125.73) (xy 133.35 125.73)
+		)
+		(stroke
+			(width 0)
+			(type default)
+		)
+	)
+	(wire
+		(pts
 			(xy 153.67 128.27) (xy 167.64 128.27)
+		)
+		(stroke
+			(width 0)
+			(type default)
+		)
+	)
+	(wire
+		(pts
+			(xy 133.35 123.19) (xy 119.38 123.19)
 		)
 		(stroke
@@
 	(symbol
 		(lib_id "power:GND")
+		(at 119.38 137.16 0)
+		(unit 1)
+		(exclude_from_sim no)
+		(in_bom yes)
+		(on_board yes)
+		(dnp no)
+		(fields_autoplaced yes)
+		(property "Reference" "#PWR02305"
+			(at 119.38 143.51 0)
+			(effects
+				(font
+					(size 1.27 1.27)
+				)
+				(hide yes)
+			)
+		)
+		(property "Value" "GND"
+			(at 119.38 142.24 0)
+			(effects
+				(font
+					(size 1.27 1.27)
+				)
+			)
+		)
+		(property "Footprint" ""
+			(at 119.38 137.16 0)
+			(effects
+				(font
+					(size 1.27 1.27)
+				)
+				(hide yes)
+			)
+		)
+		(property "Datasheet" ""
+			(at 119.38 137.16 0)
+			(effects
+				(font
+					(size 1.27 1.27)
+				)
+				(hide yes)
+			)
+		)
+		(property "Description" "Power symbol creates a global label with name \"GND\" , ground"
+			(at 119.38 137.16 0)
+			(effects
+				(font
+					(size 1.27 1.27)
+				)
+				(hide yes)
+			)
+		)
+		(pin "1"
+		)
+		(instances
+			(project ""
+				(path "/b643db5c-578e-4b48-aafc-cc4190db582a/cab17c9d-df0d-4094-9bb8-ab97cd5bdd0b"
+					(reference "#PWR02305")
+					(unit 1)
+				)
+			)
+		)
+	)
+	(symbol
+		(lib_id "power:GND")
 		(at 189.23 109.22 0)
 		(unit 1)
@@
 					(unit 1)
 				)
+			)
+		)
+	)
+	(symbol
+		(lib_id "power:PWR_FLAG")
+		(at 177.8 87.63 0)
+		(unit 1)
+		(exclude_from_sim no)
+		(in_bom yes)
+		(on_board yes)
+		(dnp no)
+		(fields_autoplaced yes)
+		(property "Reference" "#FLG02301"
+			(at 177.8 85.725 0)
+			(effects
+				(font
+					(size 1.27 1.27)
+				)
+				(hide yes)
+			)
+		)
+		(property "Value" "PWR_FLAG"
+			(at 177.8 82.55 0)
+			(effects
+				(font
+					(size 1.27 1.27)
+				)
+			)
+		)
+		(property "Footprint" ""
+			(at 177.8 87.63 0)
+			(effects
+				(font
+					(size 1.27 1.27)
+				)
+				(hide yes)
+			)
+		)
+		(property "Datasheet" "~"
+			(at 177.8 87.63 0)
+			(effects
+				(font
+					(size 1.27 1.27)
+				)
+				(hide yes)
+			)
+		)
+		(property "Description" "Special symbol for telling ERC where power comes from"
+			(at 177.8 87.63 0)
+			(effects
+				(font
+					(size 1.27 1.27)
+				)
+				(hide yes)
+			)
+		)
+		(pin "1"
+		)
+		(instances
+			(project ""
+				(path "/b643db5c-578e-4b48-aafc-cc4190db582a/cab17c9d-df0d-4094-9bb8-ab97cd5bdd0b"
+					(reference "#FLG02301")
+					(unit 1)
+				)

Commit message: new fuse and ideal diode
Parts:
- C2301: symbol dnt_global:0402,100nF -> dnt_global:0402,100nF, 16V
- JP751, JP752: footprint (none) -> Jumper:SolderJumper-2_P1.3mm_Open_RoundedPad1.0x1.5mm; symbol Jumper:SolderJumper_2_Open -> dnt_global:SolderJumper_2_Open
- U2301: value RXB6_radio_receiver -> RXB6_RXB12_radio_receiver; now not fitted; now left out of the parts list
Connections:
- net +3.3V renamed +3.3VA
- net +5V renamed +5VA
Changed lines of the file:
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@@
 	(paper "A4")
 	(junction
-		(at 167.64 87.63)
+		(at 167.64 92.71)
 		(diameter 0)
 		(color 0 0 0 0)
 	)
 	(junction
-		(at 189.23 87.63)
+		(at 189.23 92.71)
 		(diameter 0)
 		(color 0 0 0 0)
 	)
 	(junction
-		(at 177.8 87.63)
+		(at 177.8 92.71)
 		(diameter 0)
 		(color 0 0 0 0)
@@
 	(wire
 		(pts
-			(xy 177.8 87.63) (xy 189.23 87.63)
+			(xy 177.8 92.71) (xy 189.23 92.71)
 		)
 		(stroke
@@
 	(wire
 		(pts
-			(xy 201.93 95.25) (xy 201.93 87.63)
-		)
-		(stroke
-			(width 0)
-			(type default)
-		)
-	)
-	(wire
-		(pts
-			(xy 167.64 83.82) (xy 167.64 87.63)
-		)
-		(stroke
-			(width 0)
-			(type default)
-		)
-	)
-	(wire
-		(pts
-			(xy 167.64 87.63) (xy 177.8 87.63)
+			(xy 201.93 95.25) (xy 201.93 92.71)
+		)
+		(stroke
+			(width 0)
+			(type default)
+		)
+	)
+	(wire
+		(pts
+			(xy 167.64 83.82) (xy 167.64 92.71)
+		)
+		(stroke
+			(width 0)
+			(type default)
+		)
+	)
+	(wire
+		(pts
+			(xy 167.64 92.71) (xy 177.8 92.71)
 		)
 		(stroke
@@
 	(wire
 		(pts
-			(xy 201.93 87.63) (xy 189.23 87.63)
+			(xy 201.93 92.71) (xy 189.23 92.71)
 		)
 		(stroke
@@
 	(wire
 		(pts
-			(xy 201.93 102.87) (xy 201.93 109.22)
+			(xy 201.93 102.87) (xy 201.93 104.14)
 		)
 		(stroke
@@
 	(wire
 		(pts
-			(xy 189.23 102.87) (xy 189.23 109.22)
-		)
-		(stroke
-			(width 0)
-			(type default)
-		)
-	)
-	(wire
-		(pts
-			(xy 167.64 87.63) (xy 167.64 106.68)
+			(xy 189.23 102.87) (xy 189.23 104.14)
+		)
+		(stroke
+			(width 0)
+			(type default)
+		)
+	)
+	(wire
+		(pts
+			(xy 167.64 92.71) (xy 167.64 106.68)
 		)
 		(stroke
@@
 	(wire
 		(pts
-			(xy 189.23 87.63) (xy 189.23 95.25)
+			(xy 189.23 92.71) (xy 189.23 95.25)
 		)
 		(stroke
@@
 	)
 	(hierarchical_label "433_RADIO_DA"
-		(shape input)
+		(shape output)
 		(at 207.01 123.19 0)
 		(effects
@@
 	)
 	(symbol
-		(lib_id "dnt_global:0402,100nF")
+		(lib_id "dnt_global:0402,100nF, 16V")
 		(at 189.23 99.06 0)
 		(unit 1)
@@
 	(symbol
 		(lib_id "power:GND")
-		(at 189.23 109.22 0)
+		(at 189.23 104.14 0)
 		(unit 1)
 		(exclude_from_sim no)
@@
 		(fields_autoplaced yes)
 		(property "Reference" "#PWR02304"
-			(at 189.23 115.57 0)
+			(at 189.23 110.49 0)
 			(effects
 				(font
@@
 		)
 		(property "Value" "GND"
-			(at 189.23 114.3 0)
+			(at 189.23 109.22 0)
 			(effects
 				(font
@@
 		)
 		(property "Footprint" ""
-			(at 189.23 109.22 0)
+			(at 189.23 104.14 0)
 			(effects
 				(font
@@
 		)
 		(property "Datasheet" ""
-			(at 189.23 109.22 0)
+			(at 189.23 104.14 0)
 			(effects
 				(font
@@
 		)
 		(property "Description" "Power symbol creates a global label with name \"GND\" , ground"
-			(at 189.23 109.22 0)
+			(at 189.23 104.14 0)
 			(effects
 				(font
@@
 	(symbol
 		(lib_id "power:PWR_FLAG")
-		(at 177.8 87.63 0)
+		(at 177.8 92.71 0)
 		(unit 1)
 		(exclude_from_sim no)
@@
 		(fields_autoplaced yes)
 		(property "Reference" "#FLG02301"
-			(at 177.8 85.725 0)
+			(at 177.8 90.805 0)
 			(effects
 				(font
@@
 		)
 		(property "Value" "PWR_FLAG"
-			(at 177.8 82.55 0)
+			(at 177.8 87.63 0)
 			(effects
 				(font
@@
 		)
 		(property "Footprint" ""
-			(at 177.8 87.63 0)
+			(at 177.8 92.71 0)
 			(effects
 				(font
@@
 		)
 		(property "Datasheet" "~"
-			(at 177.8 87.63 0)
+			(at 177.8 92.71 0)
 			(effects
 				(font
@@
 		)
 		(property "Description" "Special symbol for telling ERC where power comes from"
-			(at 177.8 87.63 0)
+			(at 177.8 92.71 0)
 			(effects
 				(font
@@
 	)
 	(symbol
-		(lib_id "Jumper:SolderJumper_2_Open")
+		(lib_id "dnt_global:SolderJumper_2_Open")
 		(at 130.81 59.69 0)
 		(unit 1)
@@
 			)
 		)
-		(property "Footprint" ""
+		(property "Footprint" "Jumper:SolderJumper-2_P1.3mm_Open_RoundedPad1.0x1.5mm"
 			(at 130.81 59.69 0)
 			(effects
@@
 	)
 	(symbol
-		(lib_id "Jumper:SolderJumper_2_Open")
+		(lib_id "dnt_global:SolderJumper_2_Open")
 		(at 130.81 73.66 0)
 		(unit 1)
@@
 			)
 		)
-		(property "Footprint" ""
+		(property "Footprint" "Jumper:SolderJumper-2_P1.3mm_Open_RoundedPad1.0x1.5mm"
 			(at 130.81 73.66 0)
 			(effects
@@
 			)
 		)
-		(property "Value" "+5V"
+		(property "Value" "+5VA"
 			(at 83.82 49.53 0)
 			(effects
@@
 	(symbol
 		(lib_id "power:GND")
-		(at 201.93 109.22 0)
+		(at 201.93 104.14 0)
 		(unit 1)
 		(exclude_from_sim no)
@@
 		(fields_autoplaced yes)
 		(property "Reference" "#PWR02303"
-			(at 201.93 115.57 0)
+			(at 201.93 110.49 0)
 			(effects
 				(font
@@
 		)
 		(property "Value" "GND"
-			(at 201.93 114.3 0)
+			(at 201.93 109.22 0)
 			(effects
 				(font
@@
 		)
 		(property "Footprint" ""
-			(at 201.93 109.22 0)
+			(at 201.93 104.14 0)
 			(effects
 				(font
@@
 		)
 		(property "Datasheet" ""
-			(at 201.93 109.22 0)
+			(at 201.93 104.14 0)
 			(effects
 				(font
@@
 		)
 		(property "Description" "Power symbol creates a global label with name \"GND\" , ground"
-			(at 201.93 109.22 0)
+			(at 201.93 104.14 0)
 			(effects
 				(font
@@
 		(unit 1)
 		(exclude_from_sim no)
-		(in_bom yes)
+		(in_bom no)
 		(on_board yes)
-		(dnp no)
+		(dnp yes)
 		(fields_autoplaced yes)
 		(property "Reference" "U2301"
@@
 			)
 		)
-		(property "Value" "RXB6_radio_receiver"
+		(property "Value" "RXB6_RXB12_radio_receiver"
 			(at 143.51 115.57 0)
 			(effects
@@
 		)
 		(property "Footprint" "dnt:RXB6 radio receiver"
-			(at 143.764 132.842 0)
-			(effects
-				(font
-					(size 1.27 1.27)
-				)
-				(hide yes)
-			)
-		)
-		(property "Datasheet" "https://www.eeant.com/datasheet/et-rxb-12.pdf"
+			(at 143.51 136.398 0)
+			(effects
+				(font
+					(size 1.27 1.27)
+				)
+				(hide yes)
+			)
+		)
+		(property "Datasheet" ""
 			(at 191.77 137.16 0)
 			(effects
@@
 			)
 		)
-		(property "Value" "+3.3V"
+		(property "Value" "+3.3VA"
 			(at 83.82 62.23 0)
 			(effects

Commit message: x
Parts:
- removed AE2302: Antenna, symbol Device:Antenna
- added 433_ALT_DATA2: +5V, TestPoint:TestPoint_Pad_D1.0mm, symbol dnt_global:TestPoint_Pad_D1.0mm
- added J17: Conn_01x01_Pin, symbol Connector:Conn_01x01_Pin
- AE2: renamed from AE2301; now in the parts list
- U8: renamed from U2301; now in the parts list
- renumbered C754 to C28, C2301 to C29, C2302 to C30, FB2301 to FB3, JP752 to JP2, JP751 to JP3, R757 to R31
Connections:
- net at AE2.1 (A), U8.1 (ANT): now also J17.1 (Pin_1)
- net at U8.7 (DA): now also 433_ALT_DATA2.1
- no-connect marks 1 -> 0

Commit message: passes sch drc
Parts:
- J17: footprint (none) -> dnt:PinHeader_1x01_P2.54mm_Vertical; symbol Connector:Conn_01x01_Pin -> dnt_global:Conn_01x01_Socket 2.54mm
Changed lines of the file:
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@@
 	(wire
 		(pts
-			(xy 167.64 130.81) (xy 167.64 138.43)
+			(xy 167.64 130.81) (xy 167.64 139.7)
 		)
 		(stroke
@@
 	(wire
 		(pts
-			(xy 119.38 125.73) (xy 119.38 137.16)
+			(xy 119.38 125.73) (xy 119.38 139.7)
 		)
 		(stroke
@@
 	(symbol
 		(lib_id "power:GND")
-		(at 119.38 137.16 0)
+		(at 119.38 139.7 0)
 		(unit 1)
 		(exclude_from_sim no)
@@
 		(fields_autoplaced yes)
 		(property "Reference" "#PWR061"
-			(at 119.38 143.51 0)
+			(at 119.38 146.05 0)
 			(effects
 				(font
@@
 		)
 		(property "Value" "GND"
-			(at 121.92 138.4299 0)
+			(at 121.92 140.9699 0)
 			(effects
 				(font
@@
 				)
 				(justify left)
+				(hide yes)
 			)
 		)
 		(property "Footprint" ""
-			(at 119.38 137.16 0)
+			(at 119.38 139.7 0)
 			(effects
 				(font
@@
 		)
 		(property "Datasheet" ""
-			(at 119.38 137.16 0)
+			(at 119.38 139.7 0)
 			(effects
 				(font
@@
 		)
 		(property "Description" "Power symbol creates a global label with name \"GND\" , ground"
-			(at 119.38 137.16 0)
+			(at 119.38 139.7 0)
 			(effects
 				(font
@@
 		)
 		(property "Value" "GND"
-			(at 191.77 105.4099 0)
-			(effects
-				(font
-					(size 1.27 1.27)
-				)
-				(justify left)
+			(at 189.23 109.22 0)
+			(effects
+				(font
+					(size 1.27 1.27)
+				)
 			)
 		)
@@
 				)
 				(justify left)
+				(hide yes)
 			)
 		)
@@
 	)
 	(symbol
-		(lib_id "Connector:Conn_01x01_Pin")
-		(at 74.93 115.57 270)
+		(lib_id "dnt_global:Conn_01x01_Socket 2.54mm")
+		(at 74.93 115.57 90)
 		(unit 1)
 		(exclude_from_sim no)
@@
 					(size 1.27 1.27)
 				)
-				(justify left)
+				(justify right)
 			)
 		)
@@
 					(size 1.27 1.27)
 				)
-				(justify left)
-			)
-		)
-		(property "Footprint" ""
-			(at 74.93 115.57 0)
+				(justify right)
+			)
+		)
+		(property "Footprint" "dnt:PinHeader_1x01_P2.54mm_Vertical"
+			(at 69.088 115.316 0)
 			(effects
 				(font
@@
 		)
 		(property "Description" "Generic connector, single row, 01x01, script generated"
-			(at 74.93 115.57 0)
+			(at 64.77 113.284 0)
 			(effects
 				(font
@@
 				)
 				(justify left)
+				(hide yes)
 			)
 		)
@@
 	(symbol
 		(lib_id "power:GND")
-		(at 167.64 138.43 0)
+		(at 167.64 139.7 0)
 		(unit 1)
 		(exclude_from_sim no)
@@
 		(fields_autoplaced yes)
 		(property "Reference" "#PWR062"
-			(at 167.64 144.78 0)
+			(at 167.64 146.05 0)
 			(effects
 				(font
@@
 		)
 		(property "Value" "GND"
-			(at 170.18 139.6999 0)
+			(at 170.18 140.9699 0)
 			(effects
 				(font
@@
 				)
 				(justify left)
+				(hide yes)
 			)
 		)
 		(property "Footprint" ""
-			(at 167.64 138.43 0)
+			(at 167.64 139.7 0)
 			(effects
 				(font
@@
 		)
 		(property "Datasheet" ""
-			(at 167.64 138.43 0)
+			(at 167.64 139.7 0)
 			(effects
 				(font
@@
 		)
 		(property "Description" "Power symbol creates a global label with name \"GND\" , ground"
-			(at 167.64 138.43 0)
+			(at 167.64 139.7 0)
 			(effects
 				(font
@@
 		)
 		(property "Value" "+5VA"
-			(at 86.36 53.3399 0)
-			(effects
-				(font
-					(size 1.27 1.27)
-				)
-				(justify left)
+			(at 83.82 49.53 0)
+			(effects
+				(font
+					(size 1.27 1.27)
+				)
 			)
 		)
@@
 		)
 		(property "Value" "GND"
-			(at 204.47 105.4099 0)
-			(effects
-				(font
-					(size 1.27 1.27)
-				)
-				(justify left)
+			(at 201.93 109.22 0)
+			(effects
+				(font
+					(size 1.27 1.27)
+				)
 			)
 		)
@@
 		)
 		(property "Value" "+3.3VA"
-			(at 86.36 66.0399 0)
-			(effects
-				(font
-					(size 1.27 1.27)
-				)
-				(justify left)
-			)
-		)
+			(at 83.82 62.23 0)
+			(effects
+				(font
+					(size 1.27 1.27)
+				)
+			)
+		)
